File: hardware/systemboard/IOSystem.sch (KiCad schematic (older format))
At the start: 0 parts

Commit message: Finished design of system board
Parts:
- added JIN0, JIN1, JOUT0, JOUT1: Conn_01x08, symbol Connector_Generic:Conn_01x08
- added RN1: 10k, Resistor_THT:R_Array_SIP9, symbol Device:R_Network08
- added UADDR0, UADDR1, UOUT0, UOUT1: 74HC574, symbol 74xx:74LS574
- added UAND1: 74HC08, symbol 74xx:74LS08
- added UIN0, UIN1: 74HC245, symbol 74xx:74HC245
- added UINV1: 74HC04, symbol 74xx:74HC04
- added UMSEL1: 74HC138, symbol 74xx:74LS138
- added UOR1: 74HC32, symbol 74xx:74LS32
- added URAM1, URAM2, URAM3, URAM4, URAM5, URAM6, URAM7: AS6C4008, symbol Library:AS6C4008
- added UROM0: SST39SF040, symbol Library:SST39SF040
- added URSEL1: 74HC139, symbol 74xx:74LS139
Connections:
- net labels added: +5V, A10, A11, A12, A13, A14, A15, A16, A17, A18, A19, A20, A21, A8, A9, E0#, E1#, E2#, E3#, E4#, E5#, E6#, E7#, GND, OE#, WE#
- wire segments 0 -> 448
- no-connect marks 18 -> 3

Commit message: Ongoing tweaks
Connections:
- wire segments 448 -> 450
- no-connect marks 3 -> 2
Changed lines of the file:
@@
 Comment4 ""
 $EndDescr
-Text HLabel 2650 800  1    50   Input ~ 0
+Text HLabel 2550 800  1    50   Input ~ 0
 A0
-Text HLabel 2550 800  1    50   Input ~ 0
+Text HLabel 2450 800  1    50   Input ~ 0
 A1
-Text HLabel 2450 800  1    50   Input ~ 0
+Text HLabel 2350 800  1    50   Input ~ 0
 A2
-Text HLabel 2350 800  1    50   Input ~ 0
+Text HLabel 2250 800  1    50   Input ~ 0
 A3
-Text HLabel 2250 800  1    50   Input ~ 0
+Text HLabel 2150 800  1    50   Input ~ 0
 A4
-Text HLabel 2150 800  1    50   Input ~ 0
+Text HLabel 2050 800  1    50   Input ~ 0
 A5
-Text HLabel 2050 800  1    50   Input ~ 0
+Text HLabel 1950 800  1    50   Input ~ 0
 A6
-Text HLabel 1950 800  1    50   Input ~ 0
-A7
 Text HLabel 5950 800  1    50   Input ~ 0
 D0
@@
 F 3 "http://www.ti.com/lit/gpn/sn74LS574" H 5450 2350 50  0001 C CNN
 	1    5450 2350
-	0    1    1    0
-$EndComp
-$Comp
-L 74xx:74HC04 U?
-U 6 1 5FA1E5AB
-P 1950 2200
-AR Path="/5FA1E5AB" Ref="U?"  Part="6"
-AR Path="/5FA0C35A/5FA1E5AB" Ref="UINV1"  Part="6"
-F 0 "UINV1" H 1950 2517 50  0000 C CNN
-F 1 "74HC04" H 1950 2426 50  0000 C CNN
-F 2 "" H 1950 2200 50  0001 C CNN
-F 3 "http://www.nxp.com/documents/data_sheet/74HC_HCT04.pdf" H 1950 2200 50  0001 C CNN
-	6    1950 2200
 	0    1    1    0
 $EndComp
@@
 Wire Wire Line
 	2500 3200 2500 3400
-Text Label 2650 1000 1    50   ~ 0
+Text Label 2550 1000 1    50   ~ 0
 A0
-Text Label 2550 1000 1    50   ~ 0
+Text Label 2450 1000 1    50   ~ 0
 A1
-Text Label 2450 1000 1    50   ~ 0
+Text Label 2350 1000 1    50   ~ 0
 A2
-Text Label 2350 1000 1    50   ~ 0
+Text Label 2250 1000 1    50   ~ 0
 A3
-Text Label 2250 1000 1    50   ~ 0
+Text Label 2150 1000 1    50   ~ 0
 A4
-Text Label 2150 1000 1    50   ~ 0
+Text Label 2050 1000 1    50   ~ 0
 A5
-Text Label 2050 1000 1    50   ~ 0
-A6
-Wire Wire Line
-	2650 1000 2650 800
 Wire Wire Line
 	2550 1000 2550 800
@@
 Wire Wire Line
 	2050 1000 2050 800
-Text Label 5950 3050 1    50   ~ 0
+Text Label 5850 3050 1    50   ~ 0
 A7
-Text Label 5850 3050 1    50   ~ 0
+Text Label 5750 3050 1    50   ~ 0
 A8
-Text Label 5750 3050 1    50   ~ 0
+Text Label 5650 3050 1    50   ~ 0
 A9
-Text Label 5650 3050 1    50   ~ 0
+Text Label 5550 3050 1    50   ~ 0
 A10
-Text Label 5550 3050 1    50   ~ 0
+Text Label 5450 3050 1    50   ~ 0
 A11
-Text Label 5450 3050 1    50   ~ 0
+Text Label 5350 3050 1    50   ~ 0
 A12
-Text Label 5350 3050 1    50   ~ 0
+Text Label 5250 3050 1    50   ~ 0
 A13
-Text Label 5250 3050 1    50   ~ 0
+Text Label 5950 4550 1    50   ~ 0
 A14
 Wire Wire Line
-	5950 3050 5950 2850
-Wire Wire Line
 	5850 3050 5850 2850
 Wire Wire Line
@@
 Wire Wire Line
 	5250 3050 5250 2850
-Text Label 5950 4550 1    50   ~ 0
+Wire Wire Line
+	5950 4550 5950 4350
+Text Label 5850 4550 1    50   ~ 0
 A15
-Text Label 5850 4550 1    50   ~ 0
+Text Label 5750 4550 1    50   ~ 0
 A16
-Text Label 5750 4550 1    50   ~ 0
+Text Label 5650 4550 1    50   ~ 0
 A17
-Text Label 5650 4550 1    50   ~ 0
+Text Label 5550 4550 1    50   ~ 0
 A18
-Text Label 5550 4550 1    50   ~ 0
+Text Label 5450 4550 1    50   ~ 0
 A19
-Text Label 5450 4550 1    50   ~ 0
+Text Label 5350 4550 1    50   ~ 0
 A20
-Text Label 5350 4550 1    50   ~ 0
+Text Label 5250 4550 1    50   ~ 0
 A21
 Wire Wire Line
-	5950 4550 5950 4350
-Wire Wire Line
 	5850 4550 5850 4350
 Wire Wire Line
@@
 Wire Wire Line
 	5350 4550 5350 4350
+Wire Wire Line
+	5250 4550 5250 4350
 Text Label 7950 6200 1    50   ~ 0
 A0
@@
 	1    0    0    -1
 $EndComp
-Wire Wire Line
-	9050 3800 9050 3750
 $Comp
 L Library:AS6C4008 URAM2
@@
 Wire Wire Line
 	1650 3800 1650 3650
-Text Label 1650 4950 1    50   ~ 0
-A7
 Wire Wire Line
 	1950 4350 1950 4300
@@
 Connection ~ 1950 1650
 Wire Wire Line
-	1950 1650 1950 1900
-Wire Wire Line
 	1300 2650 1300 2700
 Wire Wire Line
@@
 	2200 4150 2550 4150
 Wire Wire Line
-	1950 2650 1950 2500
+	1950 2650 1950 2550
 Connection ~ 1950 2650
 Wire Wire Line
@@
 Wire Wire Line
 	950  4950 950  4800
-Wire Wire Line
-	1650 4950 1650 4800
 $Comp
 L power:GND #PWR0176
 U 1 1 61477D3C
-P 1550 4900
-F 0 "#PWR0176" H 1550 4650 50  0001 C CNN
-F 1 "GND" H 1555 4727 50  0000 C CNN
-F 2 "" H 1550 4900 50  0001 C CNN
-F 3 "" H 1550 4900 50  0001 C CNN
-	1    1550 4900
+P 1650 4900
+F 0 "#PWR0176" H 1650 4650 50  0001 C CNN
+F 1 "GND" H 1655 4727 50  0000 C CNN
+F 2 "" H 1650 4900 50  0001 C CNN
+F 3 "" H 1650 4900 50  0001 C CNN
+	1    1650 4900
 	1    0    0    -1
 $EndComp
@@
 Wire Wire Line
 	1450 4850 1450 4800
-Wire Wire Line
-	1550 4900 1550 4800
-NoConn ~ 5250 4350
+Text Label 5950 3050 1    50   ~ 0
+A6
+Wire Wire Line
+	5950 3050 5950 2850
+$Comp
+L 74xx:74HC04 UINV?
+U 6 1 6003B54E
+P 1950 2250
+AR Path="/6003B54E" Ref="UINV?"  Part="6"
+AR Path="/5FA0C35A/6003B54E" Ref="UINV1"  Part="6"
+F 0 "UINV1" H 1950 2567 50  0000 C CNN
+F 1 "74HC04" H 1950 2476 50  0000 C CNN
+F 2 "" H 1950 2250 50  0001 C CNN
+F 3 "http://www.nxp.com/documents/data_sheet/74HC_HCT04.pdf" H 1950 2250 50  0001 C CNN
+	6    1950 2250
+	0    1    1    0
+$EndComp
+Wire Wire Line
+	1950 1650 1950 1950
+Wire Wire Line
+	1650 4900 1650 4850
+Wire Wire Line
+	1650 4850 1550 4850
+Connection ~ 1650 4850
+Wire Wire Line
+	1650 4850 1650 4800
+Wire Wire Line
+	1550 4850 1550 4800
+Wire Wire Line
+	9050 3800 9050 3750
 $EndSCHEMATC

Commit message: Extend IO address range to 512 bytes. Allows to map a complete page (256 bytes) of main address range to the extended RAM.
Connections:
- net labels added: A22, A23
- wire segments 450 -> 451
Changed lines of the file:
@@
 	3900 6350 4250 6350
-Wire Wire Line
-	1950 800  1950 1100
-Wire Wire Line
-	3050 1100 1950 1100
-Connection ~ 1950 1100
-Wire Wire Line
-	1950 1100 1950 1650
 Wire Wire Line
 	3050 1650 1950 1650
@@
 Wire Wire Line
 	2050 1000 2050 800
+Text Label 5250 4550 1    50   ~ 0
+A23
+Text Label 5950 3050 1    50   ~ 0
+A8
 Text Label 5850 3050 1    50   ~ 0
-A7
+A9
 Text Label 5750 3050 1    50   ~ 0
-A8
+A10
 Text Label 5650 3050 1    50   ~ 0
-A9
+A11
 Text Label 5550 3050 1    50   ~ 0
-A10
+A12
 Text Label 5450 3050 1    50   ~ 0
-A11
+A13
 Text Label 5350 3050 1    50   ~ 0
-A12
+A14
+Wire Wire Line
+	5850 3050 5850 2850
+Wire Wire Line
+	5750 3050 5750 2850
+Wire Wire Line
+	5650 3050 5650 2850
+Wire Wire Line
+	5550 3050 5550 2850
+Wire Wire Line
+	5450 3050 5450 2850
+Wire Wire Line
+	5350 3050 5350 2850
+Wire Wire Line
+	5250 3050 5250 2850
+Wire Wire Line
+	5950 4550 5950 4350
 Text Label 5250 3050 1    50   ~ 0
-A13
+A15
 Text Label 5950 4550 1    50   ~ 0
-A14
-Wire Wire Line
-	5850 3050 5850 2850
-Wire Wire Line
-	5750 3050 5750 2850
-Wire Wire Line
-	5650 3050 5650 2850
-Wire Wire Line
-	5550 3050 5550 2850
-Wire Wire Line
-	5450 3050 5450 2850
-Wire Wire Line
-	5350 3050 5350 2850
-Wire Wire Line
-	5250 3050 5250 2850
-Wire Wire Line
-	5950 4550 5950 4350
+A16
 Text Label 5850 4550 1    50   ~ 0
-A15
+A17
 Text Label 5750 4550 1    50   ~ 0
-A16
+A18
 Text Label 5650 4550 1    50   ~ 0
-A17
+A19
 Text Label 5550 4550 1    50   ~ 0
-A18
+A20
 Text Label 5450 4550 1    50   ~ 0
-A19
-Text Label 5350 4550 1    50   ~ 0
-A20
-Text Label 5250 4550 1    50   ~ 0
 A21
 Wire Wire Line
@@
 Wire Wire Line
 	1100 1850 1100 850
-Connection ~ 1950 1650
 Wire Wire Line
 	1300 2650 1300 2700
@@
 	950  4950 950  4800
 $Comp
-L power:GND #PWR0176
-U 1 1 61477D3C
-P 1650 4900
-F 0 "#PWR0176" H 1650 4650 50  0001 C CNN
-F 1 "GND" H 1655 4727 50  0000 C CNN
-F 2 "" H 1650 4900 50  0001 C CNN
-F 3 "" H 1650 4900 50  0001 C CNN
-	1    1650 4900
-	1    0    0    -1
-$EndComp
-$Comp
 L power:+5V #PWR0177
 U 1 1 61477DA9
-P 1450 4850
-F 0 "#PWR0177" H 1450 4700 50  0001 C CNN
-F 1 "+5V" H 1465 5023 50  0000 C CNN
-F 2 "" H 1450 4850 50  0001 C CNN
-F 3 "" H 1450 4850 50  0001 C CNN
-	1    1450 4850
+P 1450 4950
+F 0 "#PWR0177" H 1450 4800 50  0001 C CNN
+F 1 "+5V" H 1465 5123 50  0000 C CNN
+F 2 "" H 1450 4950 50  0001 C CNN
+F 3 "" H 1450 4950 50  0001 C CNN
+	1    1450 4950
 	-1   0    0    1
 $EndComp
-Wire Wire Line
-	1450 4850 1450 4800
-Text Label 5950 3050 1    50   ~ 0
-A6
+Text Label 5350 4550 1    50   ~ 0
+A22
 Wire Wire Line
 	5950 3050 5950 2850
@@
 $EndComp
 Wire Wire Line
+	9050 3800 9050 3750
+Text HLabel 1850 800  1    50   Input ~ 0
+A7
+Text HLabel 1750 800  1    50   Input ~ 0
+A8
+Wire Wire Line
+	1750 1100 1750 800
+Wire Wire Line
+	1750 1100 3050 1100
+Wire Wire Line
+	1750 1100 1750 1650
+Connection ~ 1750 1100
+Wire Wire Line
 	1950 1650 1950 1950
 Wire Wire Line
-	1650 4900 1650 4850
-Wire Wire Line
-	1650 4850 1550 4850
-Connection ~ 1650 4850
-Wire Wire Line
-	1650 4850 1650 4800
-Wire Wire Line
-	1550 4850 1550 4800
-Wire Wire Line
-	9050 3800 9050 3750
+	1950 1650 1750 1650
+Connection ~ 1950 1650
+Text Label 1950 1000 1    50   ~ 0
+A6
+Text Label 1850 1000 1    50   ~ 0
+A7
+Wire Wire Line
+	1850 1000 1850 800
+Wire Wire Line
+	1950 1000 1950 800
+Text Label 1550 4950 1    50   ~ 0
+A22
+Text Label 1650 4950 1    50   ~ 0
+A23
+Wire Wire Line
+	1450 4800 1450 4950
+Wire Wire Line
+	1550 4800 1550 4950
+Wire Wire Line
+	1650 4950 1650 4800
 $EndSCHEMATC
