File: hardware/systemboard/systemboard.sch (KiCad schematic (older format))
At the start: 19 parts, among them J1 Conn_01x06, J2 Conn_01x08, J3 Conn_01x16, U1 IS61C1024AL, U2 74HC688, U3 74HC245, U4 74HC245, U5 74LS163, U6 NE555, U7 74HC74, U8 74HC04, U9 74HC32, Y1 Crystal

Commit message: Finished design of system board
Parts:
- removed unit 6 of U8
- renumbered U3 to UABUS1, U5 to UCLK1, U7 to UCLK2, U4 to UDBUS1, U1 to UFASTRAM0, U8 to UINV1, U9 to UOR2, U6 to URESET1, U2 to UZERO1
Connections:
- wire segments 260 -> 259
- no-connect marks 10 -> 9
Changed lines of the file:
@@
 U 1 1 5F982EFE
 P 7300 850
-F 0 "J1" V 7266 1130 50  0000 L CNN
-F 1 "Conn_01x06" V 7175 1130 50  0000 L CNN
+F 0 "J1" V 7500 800 50  0000 L CNN
+F 1 "Conn_01x06" V 7400 600 50  0000 L CNN
 F 2 "" H 7300 850 50  0001 C CNN
 F 3 "~" H 7300 850 50  0001 C CNN
@@
 $EndComp
 $Comp
-L 74xx:74HC245 U4
+L 74xx:74HC245 UDBUS1
 U 1 1 5FA115D2
 P 6250 3850
-F 0 "U4" V 6750 3450 50  0000 C CNN
+F 0 "UDBUS1" V 6750 3350 50  0000 C CNN
 F 1 "74HC245" V 6650 3350 50  0000 C CNN
 F 2 "" H 6250 3850 50  0001 C CNN
@@
 $EndComp
 $Comp
-L 74xx:74HC245 U3
+L 74xx:74HC245 UABUS1
 U 1 1 5FA9F853
 P 4400 3850
-F 0 "U3" V 4900 3450 50  0000 C CNN
+F 0 "UABUS1" V 4900 3450 50  0000 C CNN
 F 1 "74HC245" V 4800 3350 50  0000 C CNN
 F 2 "" H 4400 3850 50  0001 C CNN
@@
 $EndComp
 $Comp
-L 74xx:74HC04 U8
+L 74xx:74HC04 UINV1
 U 1 1 5FAD80A3
 P 9150 5050
-F 0 "U8" H 9150 5367 50  0000 C CNN
+F 0 "UINV1" H 9150 5367 50  0000 C CNN
 F 1 "74HC04" H 9150 5276 50  0000 C CNN
 F 2 "" H 9150 5050 50  0001 C CNN
@@
 $EndComp
 $Comp
-L 74xx:74HC04 U8
+L 74xx:74HC04 UINV1
 U 2 1 5FAD8137
 P 9900 5050
-F 0 "U8" H 9950 4750 50  0000 R CNN
+F 0 "UINV1" H 9950 4750 50  0000 R CNN
 F 1 "74HC04" H 10050 4850 50  0000 R CNN
 F 2 "" H 9900 5050 50  0001 C CNN
@@
 $EndComp
 $Comp
-L 74xx:74HC04 U8
+L 74xx:74HC04 UINV1
 U 3 1 5FAD8190
 P 10600 5050
-F 0 "U8" H 10600 5367 50  0000 C CNN
+F 0 "UINV1" H 10600 5367 50  0000 C CNN
 F 1 "74HC04" H 10600 5276 50  0000 C CNN
 F 2 "" H 10600 5050 50  0001 C CNN
@@
 $EndComp
 $Comp
-L 74xx:74HC04 U8
+L 74xx:74HC04 UINV1
 U 4 1 5FAD81F1
 P 8900 1450
-F 0 "U8" H 8900 1133 50  0000 C CNN
+F 0 "UINV1" H 8900 1133 50  0000 C CNN
 F 1 "74HC04" H 8900 1224 50  0000 C CNN
 F 2 "" H 8900 1450 50  0001 C CNN
@@
 $EndComp
 $Comp
-L 74xx:74HC04 U8
+L 74xx:74HC04 UINV1
 U 5 1 5FAD8258
 P 10750 3450
-F 0 "U8" H 10750 3767 50  0000 C CNN
+F 0 "UINV1" H 10750 3767 50  0000 C CNN
 F 1 "74HC04" H 10750 3676 50  0000 C CNN
 F 2 "" H 10750 3450 50  0001 C CNN
@@
 	5    10750 3450
 	0    1    1    0
-$EndComp
-$Comp
-L 74xx:74HC04 U8
-U 6 1 5FAD82C5
-P 2200 5500
-F 0 "U8" H 2200 5817 50  0000 C CNN
-F 1 "74HC04" H 2200 5726 50  0000 C CNN
-F 2 "" H 2200 5500 50  0001 C CNN
-F 3 "http://www.nxp.com/documents/data_sheet/74HC_HCT04.pdf" H 2200 5500 50  0001 C CNN
-	6    2200 5500
-	1    0    0    -1
 $EndComp
 Text Label 6450 1150 1    50   ~ 0
@@
 Connection ~ 9500 5050
 $Comp
-L 74xx:74LS74 U7
+L 74xx:74LS74 UCLK2
 U 1 1 6002F2BA
 P 7950 3900
-F 0 "U7" H 8250 4300 50  0000 R CNN
+F 0 "UCLK2" H 8250 4300 50  0000 R CNN
 F 1 "74HC74" H 8350 4200 50  0000 R CNN
 F 2 "" H 7950 3900 50  0001 C CNN
@@
 $EndComp
 $Comp
-L 74xx:74LS74 U7
+L 74xx:74LS74 UCLK2
 U 2 1 6002F327
 P 7950 2950
-F 0 "U7" H 8150 3350 50  0000 C CNN
+F 0 "UCLK2" H 8150 3350 50  0000 C CNN
 F 1 "74HC74" H 8200 3250 50  0000 C CNN
 F 2 "" H 7950 2950 50  0001 C CNN
@@
 $EndComp
 $Comp
-L 74xx:74LS74 U7
+L 74xx:74LS74 UCLK2
 U 3 1 6002F3A0
 P 900 6900
-F 0 "U7" H 1130 6946 50  0000 L CNN
+F 0 "UCLK2" H 1130 6946 50  0000 L CNN
 F 1 "74HC74" H 1130 6855 50  0000 L CNN
 F 2 "" H 900 6900 50  0001 C CNN
@@
 $EndComp
 $Comp
-L 74xx:74LS32 U9
+L 74xx:74LS32 UOR2
 U 1 1 601611CB
 P 7950 4800
-F 0 "U9" H 7950 5125 50  0000 C CNN
+F 0 "UOR2" H 7950 5125 50  0000 C CNN
 F 1 "74HC32" H 7950 5034 50  0000 C CNN
 F 2 "" H 7950 4800 50  0001 C CNN
@@
 $EndComp
 $Comp
-L 74xx:74LS32 U9
+L 74xx:74LS32 UOR2
 U 2 1 60161252
 P 5450 6750
-F 0 "U9" H 5450 7075 50  0000 C CNN
+F 0 "UOR2" H 5450 7075 50  0000 C CNN
 F 1 "74HC32" H 5450 6984 50  0000 C CNN
 F 2 "" H 5450 6750 50  0001 C CNN
@@
 $EndComp
 $Comp
-L 74xx:74LS32 U9
+L 74xx:74LS32 UOR2
 U 3 1 601612C7
 P 6000 6750
-F 0 "U9" H 6000 7075 50  0000 C CNN
+F 0 "UOR2" H 6000 7075 50  0000 C CNN
 F 1 "74HC32" H 6000 6984 50  0000 C CNN
 F 2 "" H 6000 6750 50  0001 C CNN
@@
 $EndComp
 $Comp
-L 74xx:74LS32 U9
+L 74xx:74LS32 UOR2
 U 4 1 60161340
 P 7950 2100
-F 0 "U9" H 8250 2350 50  0000 R CNN
+F 0 "UOR2" H 8250 2350 50  0000 R CNN
 F 1 "74HC32" H 8350 2250 50  0000 R CNN
 F 2 "" H 7950 2100 50  0001 C CNN
@@
 $EndComp
 $Comp
-L 74xx:74LS32 U9
+L 74xx:74LS32 UOR2
 U 5 1 601613CB
 P 2500 6900
-F 0 "U9" H 2730 6946 50  0000 L CNN
+F 0 "UOR2" H 2730 6946 50  0000 L CNN
 F 1 "74HC32" H 2730 6855 50  0000 L CNN
 F 2 "" H 2500 6900 50  0001 C CNN
@@
 $EndComp
 $Comp
-L Timer:NE555 U6
+L Timer:NE555 URESET1
 U 1 1 602470C7
 P 9750 1650
-F 0 "U6" H 9750 2228 50  0000 C CNN
+F 0 "URESET1" H 9750 2228 50  0000 C CNN
 F 1 "NE555" H 9750 2137 50  0000 C CNN
 F 2 "" H 9750 1650 50  0001 C CNN
@@
 ZEROPAGE#
 $Comp
-L Library:IS61C1024AL U1
+L Library:IS61C1024AL UFASTRAM0
 U 1 1 5F9B5E59
 P 3800 2200
-F 0 "U1" V 3900 2300 50  0000 R CNN
+F 0 "UFASTRAM0" V 3900 2600 50  0000 R CNN
 F 1 "IS61C1024AL" V 3800 2700 50  0000 R CNN
 F 2 "" H 3800 2200 50  0001 C CNN
@@
 	4700 1800 4700 1600
 $Comp
-L 74xx:74LS688 U2
+L 74xx:74LS688 UZERO1
 U 1 1 5F9831DB
 P 2050 3850
-F 0 "U2" V 2150 4950 50  0000 L CNN
+F 0 "UZERO1" V 2150 4900 50  0000 L CNN
 F 1 "74HC688" V 2250 4950 50  0000 L CNN
 F 2 "" H 2050 3850 50  0001 C CNN
@@
 $EndComp
 $Comp
-L 74xx:74LS163 U5
+L 74xx:74LS163 UCLK1
 U 1 1 600F6923
 P 9600 3450
-F 0 "U5" V 10100 3200 50  0000 R CNN
+F 0 "UCLK1" V 10100 3200 50  0000 R CNN
 F 1 "74LS163" V 10000 3250 50  0000 R CNN
 F 2 "" H 9600 3450 50  0001 C CNN
@@
 	10900 5050 10950 5050
 $Comp
-L 74xx:74HC04 U8
+L 74xx:74HC04 UINV1
 U 7 1 5FAD8334
 P 1700 6900
-F 0 "U8" H 1930 6946 50  0000 L CNN
+F 0 "UINV1" H 1930 6946 50  0000 L CNN
 F 1 "74HC04" H 1930 6855 50  0000 L CNN
 F 2 "" H 1700 6900 50  0001 C CNN
@@
 Wire Wire Line
 	1250 5950 1250 5750
-NoConn ~ 2500 5500
-$Comp
-L power:GND #PWR0137
-U 1 1 60819812
-P 1900 5550
-F 0 "#PWR0137" H 1900 5300 50  0001 C CNN
-F 1 "GND" H 1905 5377 50  0000 C CNN
-F 2 "" H 1900 5550 50  0001 C CNN
-F 3 "" H 1900 5550 50  0001 C CNN
-	1    1900 5550
-	1    0    0    -1
-$EndComp
-Wire Wire Line
-	1900 5550 1900 5500
 Wire Wire Line
 	900  6350 900  6500

Commit message: Ongoing tweaks
Parts:
- removed UCLK2: 74HC74, symbol 74xx:74LS74
- UCLK1: value 74LS163 -> 74HC163
- renumbered UFASTRAM0 to UFASTRAM1
Connections:
- net labels added: IORD#, IOWR#
- net labels removed: IO#, ZEROPAGE#
- wire segments 259 -> 243
- no-connect marks 9 -> 6
Other:
- moved on the sheet: UCLK1, UINV1A, UINV1B, UINV1C, UINV1D, UINV1E, URESET1

Commit message: Adjusting hardware to better fit 7400 parts. Small test program.
Connections:
- wire segments 243 -> 245
- no-connect marks 6 -> 7
Other:
- moved on the sheet: UINV1D

Commit message: Extend IO address range to 512 bytes. Allows to map a complete page (256 bytes) of main address range to the extended RAM.
Connections:
- wire segments 245 -> 247
- no-connect marks 7 -> 6
Changed lines of the file:
@@
 Wire Wire Line
 	900  7450 900  7400
-$Comp
-L power:+5V #PWR0104
-U 1 1 5FE06DEE
-P 3900 3350
-F 0 "#PWR0104" H 3900 3200 50  0001 C CNN
-F 1 "+5V" H 3915 3523 50  0000 C CNN
-F 2 "" H 3900 3350 50  0001 C CNN
-F 3 "" H 3900 3350 50  0001 C CNN
-	1    3900 3350
-	1    0    0    -1
-$EndComp
 Wire Wire Line
 	900  6400 900  6350
@@
 	2650 3350 2650 2800
 Connection ~ 2650 2800
-Wire Wire Line
-	2750 3350 2750 2750
-Connection ~ 2750 2750
 $Comp
 L power:GND #PWR0103
@@
 Wire Wire Line
 	3200 4700 3200 4500
-NoConn ~ 3900 4350
-Wire Wire Line
-	650  3300 1150 3300
-Wire Wire Line
-	950  3350 950  3200
-Wire Wire Line
-	950  3200 2850 3200
-Wire Wire Line
-	2850 3200 2850 2700
-Connection ~ 2850 2700
+Wire Wire Line
+	650  3300 950  3300
 Wire Wire Line
 	2550 4500 2750 4500
@@
 Wire Wire Line
 	7800 1350 9350 1350
+Text Label 7700 3200 2    50   ~ 0
+RES#
+Wire Wire Line
+	6650 2700 6800 2700
+Wire Wire Line
+	6650 2700 6650 3350
+Wire Wire Line
+	6850 3200 6750 3200
+Wire Wire Line
+	6750 3200 6750 3350
+Wire Wire Line
+	7400 2800 7400 2700
+Wire Wire Line
+	7400 2700 7400 2600
+Connection ~ 7400 2700
+Wire Wire Line
+	7400 2700 7700 2700
+Wire Wire Line
+	7450 3200 7700 3200
+Wire Wire Line
+	2950 6950 2950 7100
+Wire Wire Line
+	5000 2600 5000 3100
+Wire Wire Line
+	2050 3100 5000 3100
+Wire Wire Line
+	4900 3050 4900 2600
+Wire Wire Line
+	2150 3050 4900 3050
+Wire Wire Line
+	4800 3000 4800 2600
+Wire Wire Line
+	2250 3000 4800 3000
+Wire Wire Line
+	4700 2950 4700 2600
+Wire Wire Line
+	2350 2950 4700 2950
+Wire Wire Line
+	4600 2900 4600 2600
+Wire Wire Line
+	2450 2900 4600 2900
+Wire Wire Line
+	4500 2850 4500 2600
+Wire Wire Line
+	2550 2850 4500 2850
+Wire Wire Line
+	4400 2800 4400 2600
+Wire Wire Line
+	2650 2800 4400 2800
+Wire Wire Line
+	4300 2750 4300 2600
+Wire Wire Line
+	2750 2750 4300 2750
+Wire Wire Line
+	4200 2700 4200 2600
+Wire Wire Line
+	2850 2700 4200 2700
+Wire Wire Line
+	4100 2650 4100 2600
+Wire Wire Line
+	2950 2650 4100 2650
+Wire Wire Line
+	3750 2600 3750 2500
+Wire Wire Line
+	3750 2600 4000 2600
+Wire Wire Line
+	950  3350 950  3300
+Connection ~ 950  3300
+Wire Wire Line
+	950  3300 1150 3300
+$Comp
+L power:GND #PWR0104
+U 1 1 5FCBE6A8
+P 2800 3350
+F 0 "#PWR0104" H 2800 3100 50  0001 C CNN
+F 1 "GND" V 2805 3222 50  0000 R CNN
+F 2 "" H 2800 3350 50  0001 C CNN
+F 3 "" H 2800 3350 50  0001 C CNN
+	1    2800 3350
+	0    -1   -1   0
+$EndComp
+Wire Wire Line
+	2750 3350 2800 3350
+Text Label 3900 3200 3    50   ~ 0
+A7
+Wire Wire Line
+	3900 3350 3900 3200
 $Sheet
-S 3800 4750 2750 1600
+S 3700 4750 2850 1600
 U 5FA0C35A
 F0 "IOSystem" 50
@@
 F18 "IORD#" I B 6100 6350 50
 F19 "RES#" I B 6450 6350 50
+F20 "A7" I T 3900 4750 50
+F21 "A8" I T 3800 4750 50
 $EndSheet
-Text Label 7700 3200 2    50   ~ 0
-RES#
-Wire Wire Line
-	6650 2700 6800 2700
-Wire Wire Line
-	6650 2700 6650 3350
-Wire Wire Line
-	6850 3200 6750 3200
-Wire Wire Line
-	6750 3200 6750 3350
-Wire Wire Line
-	7400 2800 7400 2700
-Wire Wire Line
-	7400 2700 7400 2600
-Connection ~ 7400 2700
-Wire Wire Line
-	7400 2700 7700 2700
-Wire Wire Line
-	7450 3200 7700 3200
-Wire Wire Line
-	2950 6950 2950 7100
-Wire Wire Line
-	5000 2600 5000 3100
-Wire Wire Line
-	2050 3100 5000 3100
-Wire Wire Line
-	4900 3050 4900 2600
-Wire Wire Line
-	2150 3050 4900 3050
-Wire Wire Line
-	4800 3000 4800 2600
-Wire Wire Line
-	2250 3000 4800 3000
-Wire Wire Line
-	4700 2950 4700 2600
-Wire Wire Line
-	2350 2950 4700 2950
-Wire Wire Line
-	4600 2900 4600 2600
-Wire Wire Line
-	2450 2900 4600 2900
-Wire Wire Line
-	4500 2850 4500 2600
-Wire Wire Line
-	2550 2850 4500 2850
-Wire Wire Line
-	4400 2800 4400 2600
-Wire Wire Line
-	2650 2800 4400 2800
-Wire Wire Line
-	4300 2750 4300 2600
-Wire Wire Line
-	2750 2750 4300 2750
-Wire Wire Line
-	4200 2700 4200 2600
-Wire Wire Line
-	2850 2700 4200 2700
-Wire Wire Line
-	4100 2650 4100 2600
-Wire Wire Line
-	2950 2650 4100 2650
-Wire Wire Line
-	3750 2600 3750 2500
-Wire Wire Line
-	3750 2600 4000 2600
+Wire Wire Line
+	3900 4750 3900 4350
+Text Label 3800 4500 3    50   ~ 0
+A8
+Wire Wire Line
+	3800 4750 3800 4500
 $EndSCHEMATC

Commit message: Extend clock for all IO accesses - not only read access.
Connections:
- net labels added: IO#
Changed lines of the file:
@@
 $EndComp
 Text Label 9200 4450 1    50   ~ 0
-IORD#
+IO#
 Wire Wire Line
 	9400 4100 9400 4150
@@
 Wire Wire Line
 	3800 4750 3800 4500
+Text Label 2750 4450 1    50   ~ 0
+IO#
 $EndSCHEMATC

Commit message: Example program to do some serious number crunching. The machine is not running stable yet.
Parts:
- added SWRES1: SW_Push, symbol Switch:SW_Push
Connections:
- wire segments 247 -> 251
Changed lines of the file:
@@
 L power:+5V #PWR0110
 U 1 1 602EBC0B
-P 10550 900
-F 0 "#PWR0110" H 10550 750 50  0001 C CNN
-F 1 "+5V" H 10565 1073 50  0000 C CNN
-F 2 "" H 10550 900 50  0001 C CNN
-F 3 "" H 10550 900 50  0001 C CNN
-	1    10550 900
+P 10550 800
+F 0 "#PWR0110" H 10550 650 50  0001 C CNN
+F 1 "+5V" H 10565 973 50  0000 C CNN
+F 2 "" H 10550 800 50  0001 C CNN
+F 3 "" H 10550 800 50  0001 C CNN
+	1    10550 800
 	1    0    0    -1
 $EndComp
@@
 Text Label 2750 4450 1    50   ~ 0
 IO#
+$Comp
+L Switch:SW_Push SWRES1
+U 1 1 5FD5209E
+P 10950 1100
+F 0 "SWRES1" V 10700 1000 50  0000 L CNN
+F 1 "SW_Push" V 10600 1000 50  0000 L CNN
+F 2 "" H 10950 1300 50  0001 C CNN
+F 3 "" H 10950 1300 50  0001 C CNN
+	1    10950 1100
+	0    1    1    0
+$EndComp
+Wire Wire Line
+	10950 900  10550 900
+Connection ~ 10550 900
+Wire Wire Line
+	10550 900  10550 800
+Wire Wire Line
+	10950 1300 10950 1350
+Wire Wire Line
+	10950 1350 10550 1350
 $EndSCHEMATC
