File: hardware/cpuboard/Addressing.sch (KiCad schematic (older format))
At the start: 9 parts

Commit message: Simple emulator and a few more sample programs
Parts:
- UM2: value 7HCS157 -> 74HC157
Changed lines of the file:
@@
 P 5200 1250
 F 0 "UM2" V 5550 500 50  0000 L CNN
-F 1 "7HCS157" V 5650 500 50  0000 L CNN
+F 1 "74HC157" V 5650 500 50  0000 L CNN
 F 2 "" H 5200 1250 50  0001 C CNN
 F 3 "http://www.ti.com/lit/gpn/sn74LS157" H 5200 1250 50  0001 C CNN

Commit message: Add immediate addressing mode to DP instruction.
Parts:
- added UM4, UM5: 74HC157, symbol 74xx:74LS157
Connections:
- net labels added: DPI, DPI0, DPI1, DPI2
- wire segments 230 -> 266
