File: hardware/cpuboard/Control.sch (KiCad schematic (older format))
At the start: 7 parts, among them U2 74HC32, U3 74HC08, U4 74HC00, U5 74HC11

Commit message: Working on system board
Parts:
- removed unit 3 of U3
Connections:
- wire segments 155 -> 151
- no-connect marks 4 -> 3
Changed lines of the file:
@@
-$EndComp
-$Comp
-L 74xx:74LS08 U3
-U 3 1 6030F158
-P 10300 4450
-F 0 "U3" V 10350 4200 50  0000 C CNN
-F 1 "74HC08" V 10250 4100 50  0000 C CNN
-F 2 "" H 10300 4450 50  0001 C CNN
-F 3 "http://www.ti.com/lit/gpn/sn74LS08" H 10300 4450 50  0001 C CNN
-	3    10300 4450
-	1    0    0    -1
 $EndComp
 $Comp
@@
 Wire Wire Line
 	5150 4200 5400 4200
-Wire Wire Line
-	9950 4900 9950 4550
-Wire Wire Line
-	9950 4550 10000 4550
-Connection ~ 9950 4900
-Wire Wire Line
-	9950 4550 9950 4350
-Wire Wire Line
-	9950 4350 10000 4350
-Connection ~ 9950 4550
 $Comp
 L 74xx:74LS138 UDEC1
@@
 Wire Wire Line
 	2150 3550 2150 4150
-NoConn ~ 10600 4450
 NoConn ~ 2650 4150
 Wire Wire Line

Commit message: Introduce a few bit of 74AC logic parts to speed up some critical signals. Use two 74HC gates in tandem to create a more stable clock.
Parts:
- removed unit 1 of U2
- added U6: 74AC32, symbol 74xx:74LS32
- U4: value 74HC00 -> 74AC00
Connections:
- net labels added: SRESET
- wire segments 151 -> 162
- no-connect marks 3 -> 5
Other:
- moved on the sheet: U4C, U4D
Changed lines of the file:
@@
 BRANCH#
-$Comp
-L 74xx:74LS32 U2
-U 1 1 60262DE4
-P 3550 4500
-F 0 "U2" V 3650 4350 50  0000 R CNN
-F 1 "74HC32" V 3750 4450 50  0000 R CNN
-F 2 "" H 3550 4500 50  0001 C CNN
-F 3 "http://www.ti.com/lit/gpn/sn74LS32" H 3550 4500 50  0001 C CNN
-	1    3550 4500
-	0    -1   -1   0
-$EndComp
 $Comp
 L power:GND #PWR0194
@@
 P 1050 4900
 F 0 "U4" V 1050 4700 50  0000 R CNN
-F 1 "74HC00" V 950 4700 50  0000 R CNN
+F 1 "74AC00" V 950 4700 50  0000 R CNN
 F 2 "" H 1050 4900 50  0001 C CNN
 F 3 "http://www.ti.com/lit/gpn/sn74ls00" H 1050 4900 50  0001 C CNN
@@
 P 4200 4500
 F 0 "U4" V 4300 4350 50  0000 R CNN
-F 1 "74HC00" V 4400 4400 50  0000 R CNN
+F 1 "74AC00" V 4400 4400 50  0000 R CNN
 F 2 "" H 4200 4500 50  0001 C CNN
 F 3 "http://www.ti.com/lit/gpn/sn74hc00" H 4200 4500 50  0001 C CNN
@@
 	1    0    0    -1
 $EndComp
-Wire Wire Line
-	5550 1400 5600 1400
 $Comp
 L 74xx:74LS11 U5
@@
 L 74xx:74HC00 U4
 U 3 1 60354C6C
-P 10300 5000
-F 0 "U4" H 10500 5300 50  0000 C CNN
-F 1 "74HC00" H 10550 5200 50  0000 C CNN
-F 2 "" H 10300 5000 50  0001 C CNN
-F 3 "http://www.ti.com/lit/gpn/sn74hc00" H 10300 5000 50  0001 C CNN
-	3    10300 5000
+P 10750 6000
+F 0 "U4" H 10950 6300 50  0000 C CNN
+F 1 "74AC00" H 11000 6200 50  0000 C CNN
+F 2 "" H 10750 6000 50  0001 C CNN
+F 3 "http://www.ti.com/lit/gpn/sn74hc00" H 10750 6000 50  0001 C CNN
+	3    10750 6000
 	1    0    0    -1
 $EndComp
@@
 P 9850 3000
 F 0 "U4" H 10080 3046 50  0000 L CNN
-F 1 "74HC00" H 10080 2955 50  0000 L CNN
+F 1 "74AC00" H 10080 2955 50  0000 L CNN
 F 2 "" H 9850 3000 50  0001 C CNN
 F 3 "http://www.ti.com/lit/gpn/sn74hc00" H 9850 3000 50  0001 C CNN
@@
 Text HLabel 6150 5400 2    50   Input ~ 0
 PCRES#
-Wire Wire Line
-	4100 5400 4650 5400
 Connection ~ 4100 5400
 Text HLabel 6150 4200 2    50   Input ~ 0
@@
 L 74xx:74HC00 U4
 U 4 1 5FAA4DC6
-P 5250 1950
+P 5250 1850
 AR Path="/6088908D/5FAA4DC6" Ref="U4"  Part="4"
 AR Path="/60888F9A/5FAA4DC6" Ref="U?"  Part="4"
-F 0 "U4" H 5550 2200 50  0000 R CNN
-F 1 "74HC00" H 5700 2100 50  0000 R CNN
-F 2 "" H 5250 1950 50  0001 C CNN
-F 3 "http://www.ti.com/lit/gpn/sn74hc00" H 5250 1950 50  0001 C CNN
-	4    5250 1950
+F 0 "U4" H 5550 2100 50  0000 R CNN
+F 1 "74AC00" H 5700 2000 50  0000 R CNN
+F 2 "" H 5250 1850 50  0001 C CNN
+F 3 "http://www.ti.com/lit/gpn/sn74hc00" H 5250 1850 50  0001 C CNN
+	4    5250 1850
 	1    0    0    -1
 $EndComp
@@
 	1150 600  1150 750
 Wire Wire Line
-	4950 1850 4850 1850
-Wire Wire Line
-	4850 1850 4850 1650
-Wire Wire Line
-	4850 1650 5600 1650
-Wire Wire Line
-	5600 1650 5600 1400
-Connection ~ 5600 1400
-Wire Wire Line
-	5600 1400 6150 1400
-Wire Wire Line
 	3800 5400 4100 5400
 Wire Wire Line
@@
 L power:GND #PWR0182
 U 1 1 5FCCE7F2
-P 9950 5150
-F 0 "#PWR0182" H 9950 4900 50  0001 C CNN
-F 1 "GND" H 9955 4977 50  0000 C CNN
-F 2 "" H 9950 5150 50  0001 C CNN
-F 3 "" H 9950 5150 50  0001 C CNN
-	1    9950 5150
-	1    0    0    -1
-$EndComp
-Wire Wire Line
-	9950 5150 9950 5100
-Wire Wire Line
-	9950 5100 10000 5100
-Wire Wire Line
-	9950 5100 9950 4900
-Wire Wire Line
-	9950 4900 10000 4900
-Connection ~ 9950 5100
-NoConn ~ 10600 5000
+P 10400 6150
+F 0 "#PWR0182" H 10400 5900 50  0001 C CNN
+F 1 "GND" H 10405 5977 50  0000 C CNN
+F 2 "" H 10400 6150 50  0001 C CNN
+F 3 "" H 10400 6150 50  0001 C CNN
+	1    10400 6150
+	1    0    0    -1
+$EndComp
+Wire Wire Line
+	10400 6150 10400 6100
+Wire Wire Line
+	10400 6100 10450 6100
+Wire Wire Line
+	10400 6100 10400 5900
+Wire Wire Line
+	10400 5900 10450 5900
+Connection ~ 10400 6100
+NoConn ~ 11050 6000
 Text HLabel 6150 4650 2    50   Input ~ 0
 OP0
@@
 Wire Wire Line
 	1150 500  1150 600
-Wire Wire Line
-	5550 1950 7200 1950
-Connection ~ 4650 5400
-Wire Wire Line
-	4650 5400 6150 5400
-Wire Wire Line
-	4650 2050 4650 5400
-Wire Wire Line
-	4650 2050 4950 2050
 Text Label 4650 4200 1    50   ~ 0
-SRESET#
-Wire Wire Line
-	4650 2050 4650 500
-Connection ~ 4650 2050
+SRESET
 Wire Wire Line
 	7200 2450 6750 2450
@@
 	4950 2550 3550 2550
 Wire Wire Line
-	3550 2750 3550 4200
-Wire Wire Line
 	4950 3000 2350 3000
 Connection ~ 2350 3000
@@
 Connection ~ 2050 1500
 Wire Wire Line
-	2050 1500 2050 2350
+	2050 1500 2050 1950
 Wire Wire Line
 	2450 500  2450 1300
 Connection ~ 2450 1300
 Wire Wire Line
-	2450 1300 2450 2200
+	2450 1300 2450 1750
 Wire Wire Line
 	2050 500  2050 1500
+Wire Wire Line
+	4650 500  4650 2050
+Wire Wire Line
+	5550 1400 6150 1400
+Wire Wire Line
+	4000 5500 4650 5500
+Wire Wire Line
+	4650 5500 4650 5400
+Connection ~ 4000 5500
+Wire Wire Line
+	4100 5400 6150 5400
+$Comp
+L 74xx:74LS32 U6
+U 5 1 5FB6E0C9
+P 10600 4600
+F 0 "U6" H 10830 4646 50  0000 L CNN
+F 1 "74AC32" H 10830 4555 50  0000 L CNN
+F 2 "" H 10600 4600 50  0001 C CNN
+F 3 "http://www.ti.com/lit/gpn/sn74LS32" H 10600 4600 50  0001 C CNN
+	5    10600 4600
+	1    0    0    -1
+$EndComp
+$Comp
+L power:+5V #PWR0183
+U 1 1 5FB6E0CF
+P 10600 4050
+F 0 "#PWR0183" H 10600 3900 50  0001 C CNN
+F 1 "+5V" H 10615 4223 50  0000 C CNN
+F 2 "" H 10600 4050 50  0001 C CNN
+F 3 "" H 10600 4050 50  0001 C CNN
+	1    10600 4050
+	1    0    0    -1
+$EndComp
+$Comp
+L power:GND #PWR0184
+U 1 1 5FB6E0D5
+P 10600 5150
+F 0 "#PWR0184" H 10600 4900 50  0001 C CNN
+F 1 "GND" H 10605 4977 50  0000 C CNN
+F 2 "" H 10600 5150 50  0001 C CNN
+F 3 "" H 10600 5150 50  0001 C CNN
+	1    10600 5150
+	1    0    0    -1
+$EndComp
+Wire Wire Line
+	10600 5150 10600 5100
+Wire Wire Line
+	10600 4100 10600 4050
+$Comp
+L 74xx:74LS32 U6
+U 3 1 5FB897E1
+P 9650 5500
+F 0 "U6" H 9750 5800 50  0000 C CNN
+F 1 "74AC32" H 9800 5700 50  0000 C CNN
+F 2 "" H 9650 5500 50  0001 C CNN
+F 3 "http://www.ti.com/lit/gpn/sn74LS32" H 9650 5500 50  0001 C CNN
+	3    9650 5500
+	1    0    0    -1
+$EndComp
+$Comp
+L 74xx:74LS32 U6
+U 4 1 5FB897E7
+P 6150 1950
+AR Path="/6088908D/5FB897E7" Ref="U6"  Part="4"
+AR Path="/60888F9A/5FB897E7" Ref="U?"  Part="4"
+F 0 "U6" H 6300 1800 50  0000 C CNN
+F 1 "74AC32" H 6350 1700 50  0000 C CNN
+F 2 "" H 6150 1950 50  0001 C CNN
+F 3 "http://www.ti.com/lit/gpn/sn74LS32" H 6150 1950 50  0001 C CNN
+	4    6150 1950
+	1    0    0    1
+$EndComp
+$Comp
+L 74xx:74LS32 U6
+U 1 1 5FB9058F
+P 3550 4500
+F 0 "U6" H 3800 4750 50  0000 R CNN
+F 1 "74AC32" H 3950 4650 50  0000 R CNN
+F 2 "" H 3550 4500 50  0001 C CNN
+F 3 "http://www.ti.com/lit/gpn/sn74LS32" H 3550 4500 50  0001 C CNN
+	1    3550 4500
+	0    -1   -1   0
+$EndComp
+$Comp
+L 74xx:74LS32 U6
+U 2 1 5FB9733B
+P 9650 6000
+AR Path="/6088908D/5FB9733B" Ref="U6"  Part="2"
+AR Path="/60888F9A/5FB9733B" Ref="U?"  Part="2"
+F 0 "U6" H 9800 6300 50  0000 C CNN
+F 1 "74AC32" H 9850 6200 50  0000 C CNN
+F 2 "" H 9650 6000 50  0001 C CNN
+F 3 "http://www.ti.com/lit/gpn/sn74LS32" H 9650 6000 50  0001 C CNN
+	2    9650 6000
+	1    0    0    1
+$EndComp
+Wire Wire Line
+	4950 1750 2450 1750
+Connection ~ 2450 1750
+Wire Wire Line
+	2450 1750 2450 2200
+Wire Wire Line
+	4950 1950 2050 1950
+Connection ~ 2050 1950
+Wire Wire Line
+	2050 1950 2050 2350
+Wire Wire Line
+	5850 1850 5550 1850
+Wire Wire Line
+	4650 2050 5850 2050
+Wire Wire Line
+	6450 1950 7200 1950
+Connection ~ 4650 2050
+Wire Wire Line
+	4650 2050 4650 5400
+Wire Wire Line
+	3550 2750 3550 4200
+$Comp
+L power:GND #PWR0203
+U 1 1 5FBDDE97
+P 9300 6150
+F 0 "#PWR0203" H 9300 5900 50  0001 C CNN
+F 1 "GND" H 9305 5977 50  0000 C CNN
+F 2 "" H 9300 6150 50  0001 C CNN
+F 3 "" H 9300 6150 50  0001 C CNN
+	1    9300 6150
+	1    0    0    -1
+$EndComp
+$Comp
+L power:GND #PWR0204
+U 1 1 5FBDDF29
+P 9300 5650
+F 0 "#PWR0204" H 9300 5400 50  0001 C CNN
+F 1 "GND" H 9305 5477 50  0000 C CNN
+F 2 "" H 9300 5650 50  0001 C CNN
+F 3 "" H 9300 5650 50  0001 C CNN
+	1    9300 5650
+	1    0    0    -1
+$EndComp
+Wire Wire Line
+	9300 6150 9300 6100
+Wire Wire Line
+	9300 6100 9350 6100
+Wire Wire Line
+	9300 6100 9300 5900
+Wire Wire Line
+	9300 5900 9350 5900
+Connection ~ 9300 6100
+Wire Wire Line
+	9300 5650 9300 5600
+Wire Wire Line
+	9300 5600 9350 5600
+Wire Wire Line
+	9300 5600 9300 5400
+Wire Wire Line
+	9300 5400 9350 5400
+Connection ~ 9300 5600
+NoConn ~ 9950 5500
+NoConn ~ 9950 6000
 $EndSCHEMATC

Commit message: Change CPU control to only use HC parts while not losing speed. It is still possible to run at 11MHz.
Parts:
- removed U6: 74AC32, symbol 74xx:74LS32
- added U6: 74HC153, symbol 74xx:74LS153
- U4: value 74AC00 -> 74HC00
Connections:
- net labels removed: SRESET
- wire segments 162 -> 165
Other:
- moved on the sheet: U4C, U4D
