File: hardware/cpuboard/cpuboard.sch (KiCad schematic (older format))
At the start: 5 parts, among them J1 Conn_01x06, J2 Conn_01x17, J3 Conn_01x08, U1 7400

Commit message: Working on system board
Parts:
- added U3: 74HC08, symbol 74xx:74LS08
Connections:
- net labels added: CIN
- wire segments 243 -> 251
- no-connect marks 2 -> 3
Other:
- note added: "Add a 100nF ceramic \ncapacitor to every IC\nto please the gods of\nsignal integrity."
- note removed: "Add a 100nF ceramic \ncapacitor to every IC."
- moved on the sheet: U1A, U1B, U1C, U1D
Changed lines of the file:
@@
 	10800 6000 10800 6050
 Connection ~ 10800 6000
-Text Notes 10250 5200 0    50   ~ 0
-Add a 100nF ceramic \ncapacitor to every IC.
+Text Notes 10250 5300 0    50   ~ 0
+Add a 100nF ceramic \ncapacitor to every IC\nto please the gods of\nsignal integrity.
 Wire Wire Line
 	1450 5750 2000 5750
@@
 L 74xx:7400 U1
 U 1 1 5FAC566C
-P 1150 1300
-F 0 "U1" H 1350 1550 50  0000 C CNN
-F 1 "7400" H 1400 1450 50  0000 C CNN
-F 2 "" H 1150 1300 50  0001 C CNN
-F 3 "http://www.ti.com/lit/gpn/sn7400" H 1150 1300 50  0001 C CNN
-	1    1150 1300
+P 10600 2300
+F 0 "U1" H 10800 2550 50  0000 C CNN
+F 1 "7400" H 10850 2450 50  0000 C CNN
+F 2 "" H 10600 2300 50  0001 C CNN
+F 3 "http://www.ti.com/lit/gpn/sn7400" H 10600 2300 50  0001 C CNN
+	1    10600 2300
 	1    0    0    -1
 $EndComp
@@
 L 74xx:7400 U1
 U 2 1 5FAC56A9
-P 6500 1150
-F 0 "U1" H 6650 1450 50  0000 C CNN
-F 1 "7400" H 6650 1350 50  0000 C CNN
-F 2 "" H 6500 1150 50  0001 C CNN
-F 3 "http://www.ti.com/lit/gpn/sn7400" H 6500 1150 50  0001 C CNN
-	2    6500 1150
+P 10600 2850
+F 0 "U1" H 10750 3150 50  0000 C CNN
+F 1 "7400" H 10750 3050 50  0000 C CNN
+F 2 "" H 10600 2850 50  0001 C CNN
+F 3 "http://www.ti.com/lit/gpn/sn7400" H 10600 2850 50  0001 C CNN
+	2    10600 2850
 	1    0    0    -1
 $EndComp
@@
 Wire Wire Line
 	1450 1300 1600 1300
-Wire Wire Line
-	850  850  850  1200
-Wire Wire Line
-	850  1200 850  1400
-Connection ~ 850  1200
 Wire Wire Line
 	9650 5550 9650 6350
@@
 L 74xx:7400 U1
 U 3 1 5FECED65
-P 10600 2750
+P 6500 1150
 AR Path="/5FECED65" Ref="U1"  Part="3"
 AR Path="/60888F9A/5FECED65" Ref="U?"  Part="3"
-F 0 "U1" H 10600 3075 50  0000 C CNN
-F 1 "7400" H 10600 2984 50  0000 C CNN
-F 2 "" H 10600 2750 50  0001 C CNN
-F 3 "http://www.ti.com/lit/gpn/sn7400" H 10600 2750 50  0001 C CNN
-	3    10600 2750
+F 0 "U1" H 6500 1475 50  0000 C CNN
+F 1 "7400" H 6500 1384 50  0000 C CNN
+F 2 "" H 6500 1150 50  0001 C CNN
+F 3 "http://www.ti.com/lit/gpn/sn7400" H 6500 1150 50  0001 C CNN
+	3    6500 1150
 	1    0    0    -1
 $EndComp
@@
 L 74xx:7400 U1
 U 4 1 5FECED6C
-P 10600 3300
+P 10600 3400
 AR Path="/5FECED6C" Ref="U1"  Part="4"
 AR Path="/60888F9A/5FECED6C" Ref="U?"  Part="4"
-F 0 "U1" H 10800 3550 50  0000 C CNN
-F 1 "7400" H 10800 3450 50  0000 C CNN
-F 2 "" H 10600 3300 50  0001 C CNN
-F 3 "http://www.ti.com/lit/gpn/sn7400" H 10600 3300 50  0001 C CNN
-	4    10600 3300
-	1    0    0    -1
-$EndComp
-NoConn ~ 10900 2750
-NoConn ~ 10900 3300
-$Comp
-L power:GND #PWR0181
-U 1 1 5FEFA9A6
-P 10250 3500
-F 0 "#PWR0181" H 10250 3250 50  0001 C CNN
-F 1 "GND" H 10255 3327 50  0000 C CNN
-F 2 "" H 10250 3500 50  0001 C CNN
-F 3 "" H 10250 3500 50  0001 C CNN
-	1    10250 3500
-	1    0    0    -1
-$EndComp
-Wire Wire Line
-	10250 3500 10250 3400
-Wire Wire Line
-	10250 3400 10300 3400
-Wire Wire Line
-	10250 3400 10250 3200
-Wire Wire Line
-	10250 3200 10300 3200
-Connection ~ 10250 3400
-Wire Wire Line
-	10250 3200 10250 2850
-Wire Wire Line
-	10250 2850 10300 2850
-Connection ~ 10250 3200
-Wire Wire Line
-	10250 2850 10250 2650
-Wire Wire Line
-	10250 2650 10300 2650
-Connection ~ 10250 2850
+F 0 "U1" H 10800 3650 50  0000 C CNN
+F 1 "7400" H 10800 3550 50  0000 C CNN
+F 2 "" H 10600 3400 50  0001 C CNN
+F 3 "http://www.ti.com/lit/gpn/sn7400" H 10600 3400 50  0001 C CNN
+	4    10600 3400
+	1    0    0    -1
+$EndComp
 $Comp
 L Connector_Generic:Conn_01x06 J1
@@
 	0    1    -1   0
 $EndComp
+Text Label 850  1050 1    50   ~ 0
+CIN
+Wire Wire Line
+	850  1050 850  850
+Wire Wire Line
+	10250 2200 10250 2400
+Wire Wire Line
+	10250 2400 10300 2400
+Wire Wire Line
+	10250 2200 10300 2200
+Wire Wire Line
+	10250 2400 10250 2750
+Wire Wire Line
+	10250 2750 10300 2750
+Connection ~ 10250 2400
+Wire Wire Line
+	10250 2750 10250 2950
+Wire Wire Line
+	10250 2950 10300 2950
+Connection ~ 10250 2750
+Wire Wire Line
+	10250 2950 10250 3300
+Wire Wire Line
+	10250 3300 10300 3300
+Connection ~ 10250 2950
+Wire Wire Line
+	10250 3300 10250 3500
+Wire Wire Line
+	10250 3500 10300 3500
+Connection ~ 10250 3300
+Text Label 11050 4400 2    50   ~ 0
+CLK
+$Comp
+L 74xx:74LS08 U?
+U 3 1 5F9E78CE
+P 10600 4400
+AR Path="/6088908D/5F9E78CE" Ref="U?"  Part="3"
+AR Path="/5F9E78CE" Ref="U3"  Part="3"
+F 0 "U3" H 10850 4550 50  0000 C CNN
+F 1 "74HC08" H 10850 4650 50  0000 C CNN
+F 2 "" H 10600 4400 50  0001 C CNN
+F 3 "http://www.ti.com/lit/gpn/sn74LS08" H 10600 4400 50  0001 C CNN
+	3    10600 4400
+	1    0    0    -1
+$EndComp
+Text Label 10050 4400 0    50   ~ 0
+CIN
+Wire Wire Line
+	10050 4400 10250 4400
+Wire Wire Line
+	10250 4400 10250 4500
+Wire Wire Line
+	10250 4500 10300 4500
+Wire Wire Line
+	10250 4400 10250 4300
+Wire Wire Line
+	10250 4300 10300 4300
+Connection ~ 10250 4400
+Wire Wire Line
+	10900 4400 11050 4400
+NoConn ~ 10900 2300
+NoConn ~ 10900 2850
+NoConn ~ 10900 3400
+$Comp
+L power:GND #PWR0181
+U 1 1 5FA9B133
+P 10250 3500
+F 0 "#PWR0181" H 10250 3250 50  0001 C CNN
+F 1 "GND" H 10255 3327 50  0000 C CNN
+F 2 "" H 10250 3500 50  0001 C CNN
+F 3 "" H 10250 3500 50  0001 C CNN
+	1    10250 3500
+	1    0    0    -1
+$EndComp
+Connection ~ 10250 3500
 $EndSCHEMATC

Commit message: Introduce a few bit of 74AC logic parts to speed up some critical signals. Use two 74HC gates in tandem to create a more stable clock.
Parts:
- added U2: 74HC32, symbol 74xx:74LS32
Connections:
- wire segments 251 -> 259
Changed lines of the file:
@@
 	10250 3500 10300 3500
 Connection ~ 10250 3300
-Text Label 11050 4400 2    50   ~ 0
+Text Label 11100 4300 2    50   ~ 0
 CLK
 $Comp
 L 74xx:74LS08 U?
 U 3 1 5F9E78CE
-P 10600 4400
+P 10450 4600
 AR Path="/6088908D/5F9E78CE" Ref="U?"  Part="3"
 AR Path="/5F9E78CE" Ref="U3"  Part="3"
-F 0 "U3" H 10850 4550 50  0000 C CNN
-F 1 "74HC08" H 10850 4650 50  0000 C CNN
-F 2 "" H 10600 4400 50  0001 C CNN
-F 3 "http://www.ti.com/lit/gpn/sn74LS08" H 10600 4400 50  0001 C CNN
-	3    10600 4400
+F 0 "U3" H 10700 4750 50  0000 C CNN
+F 1 "74HC08" H 10700 4850 50  0000 C CNN
+F 2 "" H 10450 4600 50  0001 C CNN
+F 3 "http://www.ti.com/lit/gpn/sn74LS08" H 10450 4600 50  0001 C CNN
+	3    10450 4600
 	1    0    0    -1
 $EndComp
-Text Label 10050 4400 0    50   ~ 0
+Text Label 9900 4350 0    50   ~ 0
 CIN
 Wire Wire Line
-	10050 4400 10250 4400
+	10100 4700 10150 4700
 Wire Wire Line
-	10250 4400 10250 4500
+	10100 4500 10150 4500
 Wire Wire Line
-	10250 4500 10300 4500
-Wire Wire Line
-	10250 4400 10250 4300
-Wire Wire Line
-	10250 4300 10300 4300
-Connection ~ 10250 4400
-Wire Wire Line
-	10900 4400 11050 4400
+	10750 4600 10900 4600
 NoConn ~ 10900 2300
 NoConn ~ 10900 2850
@@
 $EndComp
 Connection ~ 10250 3500
+$Comp
+L 74xx:74LS32 U?
+U 1 1 5FC191A6
+P 10450 4050
+AR Path="/6088908D/5FC191A6" Ref="U?"  Part="1"
+AR Path="/5FC191A6" Ref="U2"  Part="1"
+F 0 "U2" H 10700 4300 50  0000 R CNN
+F 1 "74HC32" H 10850 4200 50  0000 R CNN
+F 2 "" H 10450 4050 50  0001 C CNN
+F 3 "http://www.ti.com/lit/gpn/sn74LS32" H 10450 4050 50  0001 C CNN
+	1    10450 4050
+	1    0    0    -1
+$EndComp
+Wire Wire Line
+	10100 4500 10100 4350
+Wire Wire Line
+	10100 4150 10150 4150
+Connection ~ 10100 4500
+Wire Wire Line
+	10100 4150 10100 3950
+Wire Wire Line
+	10100 3950 10150 3950
+Connection ~ 10100 4150
+Wire Wire Line
+	10900 4600 10900 4300
+Wire Wire Line
+	10900 4050 10750 4050
+Wire Wire Line
+	11100 4300 10900 4300
+Connection ~ 10900 4300
+Wire Wire Line
+	10900 4300 10900 4050
+Wire Wire Line
+	10100 4500 10100 4700
+Wire Wire Line
+	9900 4350 10100 4350
+Connection ~ 10100 4350
+Wire Wire Line
+	10100 4350 10100 4150
 $EndSCHEMATC

Commit message: Add immediate addressing mode to DP instruction.
Parts:
- removed J2: Conn_01x17, symbol Connector_Generic:Conn_01x17
- removed U1: 7400, symbol 74xx:7400
- added J2: Conn_01x16, symbol Connector_Generic:Conn_01x16
Connections:
- wire segments 259 -> 248
- no-connect marks 3 -> 0
