File: hardware/mainboard/mainboard.sch (KiCad schematic (older format))
At the start: 31 parts, among them U1 74HC04, U2 AS6C4008, U3 74AC32, U4 74AC00, U5 SST39SF040, U7 74HC245, U9 74HC574

Commit message: Redesign memory/io interface for easier wireing on the breadboard. This also uses less ICs.
Parts:
- removed C1, C10, C11, C13, C6, C8, C9: 100nF, Capacitor_THT:C_Disc_D3.8mm_W2.6mm_P2.50mm, symbol Device:C_Small
- removed U1: 74HC04, Package_DIP:DIP-14_W7.62mm_Socket, symbol 74xx:74HC04
- removed U3: 74AC32, Package_DIP:DIP-14_W7.62mm_Socket, symbol 74xx:74LS32
- removed unit 4 of U4
- removed U7: 74HC245, Package_DIP:DIP-20_W7.62mm_Socket, symbol 74xx:74HC245
- removed U9: 74HC574, Package_DIP:DIP-20_W7.62mm_Socket, symbol 74xx:74HCT574
- removed U?: 74LS574, symbol 74xx:74LS574
- added U?: 74HC541, symbol 74xx:74LS541
- added U?: 74LS377, symbol 74xx:74LS377
- added U?: 74HC377, symbol 74xx:74LS377
- U4: value 74AC00 -> 74HC00
- gave numbers to parts that had none: 1
- renumbered D7 to LED0, D6 to LED1, D5 to LED2, D4 to LED3, D3 to LED4, D2 to LED5, D1 to LED6, D0 to LED7
Connections:
- net labels added: B0, B1, B2, B3, B4, B5, B6, B7, IOSEL#, RAMSEL#, ROMSEL#
- net labels removed: A10, A11, A12, A13, A14, A15, A8, A9, CPOUTPUT, IOMODE, OEINPUT, OERAM, OEROM, RAM, RESETIO, ROM
- wire segments 271 -> 221
- no-connect marks 4 -> 3
Other:
- note added: "DECODE"
- note removed: "MODE\nREGISTER"
- moved on the sheet: U4A, U4B, U4C, U4E
