File: hardware/mainboard/mainboard.sch (KiCad schematic (older format))
At the start: 22 parts, among them U2 AS6C4008, U4 74HC00, U5 SST39SF040

Commit message: Restructure memory map for easier compatibility with other designs
Parts:
- added unit 4 of U4
Connections:
- wire segments 221 -> 227
Other:
- moved on the sheet: U4A, U4B, U4C
Changed lines of the file:
@@
 Text Label 8000 2050 3    50   ~ 0
 A18
-Text Label 7150 3250 1    50   ~ 0
+Text Label 6750 3050 1    50   ~ 0
 RAMSEL#
 $Comp
@@
 L 74xx:7400 U4
 U 1 1 5ECCC932
-P 6000 1950
-F 0 "U4" H 6000 2275 50  0000 C CNN
-F 1 "74HC00" H 6000 2184 50  0000 C CNN
-F 2 "Package_DIP:DIP-14_W7.62mm_Socket" H 6000 1950 50  0001 C CNN
-F 3 "http://www.ti.com/lit/gpn/sn7400" H 6000 1950 50  0001 C CNN
-	1    6000 1950
-	-1   0    0    1
+P 6100 2350
+F 0 "U4" H 6100 2550 50  0000 C CNN
+F 1 "74HC00" H 6050 2650 50  0000 C CNN
+F 2 "Package_DIP:DIP-14_W7.62mm_Socket" H 6100 2350 50  0001 C CNN
+F 3 "http://www.ti.com/lit/gpn/sn7400" H 6100 2350 50  0001 C CNN
+	1    6100 2350
+	0    1    1    0
 $EndComp
 Text Label 7950 4450 1    50   ~ 0
@@
 L 74xx:7400 U4
 U 2 1 5ECE311F
-P 5550 2550
-F 0 "U4" H 5550 2875 50  0000 C CNN
-F 1 "74HC00" H 5550 2784 50  0000 C CNN
-F 2 "Package_DIP:DIP-14_W7.62mm_Socket" H 5550 2550 50  0001 C CNN
-F 3 "http://www.ti.com/lit/gpn/sn7400" H 5550 2550 50  0001 C CNN
-	2    5550 2550
+P 6750 2350
+F 0 "U4" H 6750 2675 50  0000 C CNN
+F 1 "74HC00" H 6750 2584 50  0000 C CNN
+F 2 "Package_DIP:DIP-14_W7.62mm_Socket" H 6750 2350 50  0001 C CNN
+F 3 "http://www.ti.com/lit/gpn/sn7400" H 6750 2350 50  0001 C CNN
+	2    6750 2350
 	0    -1   1    0
 $EndComp
@@
 L 74xx:7400 U4
 U 3 1 5ECE31C6
-P 6600 2550
-F 0 "U4" H 6600 2875 50  0000 C CNN
-F 1 "74HC00" H 6600 2784 50  0000 C CNN
-F 2 "Package_DIP:DIP-14_W7.62mm_Socket" H 6600 2550 50  0001 C CNN
-F 3 "http://www.ti.com/lit/gpn/sn7400" H 6600 2550 50  0001 C CNN
-	3    6600 2550
-	0    1    1    0
+P 7250 1450
+F 0 "U4" H 7250 1150 50  0000 C CNN
+F 1 "74HC00" H 7250 1250 50  0000 C CNN
+F 2 "Package_DIP:DIP-14_W7.62mm_Socket" H 7250 1450 50  0001 C CNN
+F 3 "http://www.ti.com/lit/gpn/sn7400" H 7250 1450 50  0001 C CNN
+	3    7250 1450
+	-1   0    0    1
 $EndComp
 Text Label 6200 5850 1    50   ~ 0
@@
 Wire Wire Line
 	7800 3400 7800 3250
-Text Label 6600 3250 1    50   ~ 0
+Text Label 6100 3050 1    50   ~ 0
 IOSEL#
-Wire Wire Line
-	6700 2250 6700 1950
-Wire Wire Line
-	6350 1950 6350 2050
-Wire Wire Line
-	6350 2050 6300 2050
-Wire Wire Line
-	6350 1950 6350 1850
-Wire Wire Line
-	6350 1850 6300 1850
-Connection ~ 6350 1950
-Text Label 5550 3250 1    50   ~ 0
+Text Label 5550 3050 1    50   ~ 0
 ROMSEL#
 Wire Wire Line
-	6500 1650 6500 2250
-Wire Wire Line
-	6700 1950 7150 1950
-Wire Wire Line
-	5550 2850 5550 3250
-Wire Wire Line
-	6600 2850 6600 3250
-Wire Wire Line
-	7150 3250 7150 1950
-Connection ~ 7150 1950
-Text Notes 7600 1179 2    79   ~ 0
+	6750 2650 6750 3050
+Text Notes 7000 1000 2    79   ~ 0
 DECODE
 $Comp
@@
 	3100 3250 3100 3650
 Wire Wire Line
-	8400 1950 8400 2250
-Wire Wire Line
-	8500 1650 8500 2250
-Wire Wire Line
-	7150 1950 8400 1950
-Wire Wire Line
-	6500 1650 8500 1650
-Wire Wire Line
 	7800 2250 7800 2050
 Wire Wire Line
@@
 NoConn ~ 8300 2250
 Wire Wire Line
-	6350 1950 6700 1950
-Connection ~ 6700 1950
-Wire Wire Line
-	6500 1650 5450 1650
-Wire Wire Line
-	5450 1650 5450 2250
-Connection ~ 6500 1650
-Wire Wire Line
-	5700 1950 5650 1950
-Wire Wire Line
-	5650 1950 5650 2250
+	7550 1800 7600 1800
+Wire Wire Line
+	7600 1800 7600 1900
+Wire Wire Line
+	7600 2000 7550 2000
+Wire Wire Line
+	7600 1900 8400 1900
+Wire Wire Line
+	8400 1900 8400 2250
+Connection ~ 7600 1900
+Wire Wire Line
+	7600 1900 7600 2000
+$Comp
+L 74xx:7400 U4
+U 4 1 6094D119
+P 7250 1900
+F 0 "U4" H 7250 2150 50  0000 C CNN
+F 1 "74HC00" H 7250 2250 50  0000 C CNN
+F 2 "" H 7250 1900 50  0001 C CNN
+F 3 "http://www.ti.com/lit/gpn/sn7400" H 7250 1900 50  0001 C CNN
+	4    7250 1900
+	-1   0    0    1
+$EndComp
+Wire Wire Line
+	6100 3050 6100 2650
+Wire Wire Line
+	6950 1900 6850 1900
+Wire Wire Line
+	6850 1900 6850 2050
+Wire Wire Line
+	7550 1550 7600 1550
+Wire Wire Line
+	7600 1550 7600 1450
+Wire Wire Line
+	7600 1350 7550 1350
+Wire Wire Line
+	7600 1450 8500 1450
+Wire Wire Line
+	8500 1450 8500 2250
+Connection ~ 7600 1450
+Wire Wire Line
+	7600 1450 7600 1350
+Wire Wire Line
+	6950 1450 6650 1450
+Wire Wire Line
+	6000 1450 6000 2050
+Connection ~ 6650 1450
+Wire Wire Line
+	6650 1450 6000 1450
+Wire Wire Line
+	5550 1450 6000 1450
+Connection ~ 6000 1450
+Wire Wire Line
+	8400 1900 8400 1700
+Wire Wire Line
+	8400 1700 6200 1700
+Wire Wire Line
+	6200 1700 6200 2050
+Connection ~ 8400 1900
+Wire Wire Line
+	6650 2050 6650 1450
+Wire Wire Line
+	5550 1450 5550 3050
 $EndSCHEMATC

Commit message: Change address latch interface and software access. Refactor large parts of Bernd to work with new latch interface and make code more compact also.
Parts:
- removed JCTR: Conn_01x03, symbol Connector_Generic:Conn_01x03
- added JCTR: Conn_01x05, symbol Connector_Generic:Conn_01x05
Connections:
- net labels added: CLK, LATCHA#, LATCHB#
- net labels removed: WRX#
- wire segments 227 -> 229
Changed lines of the file:
@@
 Text Label 10400 1700 2    50   ~ 0
 WR#
-Text Label 10400 1900 2    50   ~ 0
+Text Label 10400 1800 2    50   ~ 0
 RD#
 Text Label 7650 5900 1    50   ~ 0
@@
 $EndComp
 $Comp
-L Connector_Generic:Conn_01x03 JCTR
-U 1 1 60894DE5
-P 10750 1800
-F 0 "JCTR" H 10670 1475 50  0000 C CNN
-F 1 "Conn_01x03" H 10670 1566 50  0000 C CNN
-F 2 "" H 10750 1800 50  0001 C CNN
-F 3 "~" H 10750 1800 50  0001 C CNN
-	1    10750 1800
-	1    0    0    1
-$EndComp
-$Comp
 L power:PWR_FLAG #FLG?
 U 1 1 608AA4DE
@@
 Wire Wire Line
 	6200 7450 6300 7450
-Text Label 10400 1800 2    50   ~ 0
-WRX#
 Wire Wire Line
 	10550 1700 10400 1700
 Wire Wire Line
 	10550 1800 10400 1800
-Wire Wire Line
-	10550 1900 10400 1900
 Wire Wire Line
 	10550 2500 10400 2500
@@
 NoConn ~ 8200 2250
 Text Label 8700 3550 1    50   ~ 0
-WRX#
-$Comp
-L power:GND #PWR?
-U 1 1 60D49D16
-P 8800 3300
-F 0 "#PWR?" H 8800 3050 50  0001 C CNN
-F 1 "GND" V 8805 3172 50  0000 R CNN
-F 2 "" H 8800 3300 50  0001 C CNN
-F 3 "" H 8800 3300 50  0001 C CNN
-	1    8800 3300
-	1    0    0    -1
-$EndComp
-Wire Wire Line
-	8800 3300 8800 3250
+CLK
 Wire Wire Line
 	8700 3550 8700 3250
@@
 Wire Wire Line
 	5550 1450 5550 3050
+$Comp
+L Connector_Generic:Conn_01x05 JCTR
+U 1 1 6093C414
+P 10750 1900
+F 0 "JCTR" H 10650 2350 50  0000 L CNN
+F 1 "Conn_01x05" H 10550 2250 50  0000 L CNN
+F 2 "" H 10750 1900 50  0001 C CNN
+F 3 "~" H 10750 1900 50  0001 C CNN
+	1    10750 1900
+	1    0    0    -1
+$EndComp
+Text Label 10400 2000 2    50   ~ 0
+LATCHB#
+Text Label 10400 1900 2    50   ~ 0
+LATCHA#
+Text Label 10400 2100 2    50   ~ 0
+CLK
+Wire Wire Line
+	10400 1900 10550 1900
+Wire Wire Line
+	10400 2000 10550 2000
+Wire Wire Line
+	10400 2100 10550 2100
+Text Label 8800 3550 1    50   ~ 0
+LATCHB#
+Wire Wire Line
+	8800 3550 8800 3250
 $EndSCHEMATC
