File: hardware/controllerboard/controllerboard.sch (KiCad schematic (older format))
At the start: 29 parts, among them U1 74HC04, U2 74HC32, Y1 Crystal

Commit message: Modify wiring to for convenient breadboarding
Parts:
- removed unit 1 of U1
- removed unit 2 of U1
- removed unit 3 of U1
- removed unit 1 of URES1
- removed unit 2 of URES1
- added unit 4 of UCLK1
- added unit 5 of UCLK1
- added unit 6 of UCLK1
- added unit 1 of URES1
- renumbered UB1 to UA1, UA1 to UB1, U1 to UCLK1, UEQ1 to UCMP1, U2 to UOR1
Connections:
- net labels added: CMD0, CMD1, CMD2, CMDSET#, RES2
- net labels removed: CMDST#
- wire segments 480 -> 462
- no-connect marks 11 -> 9

Commit message: Rework tooling for new architecture
Connections:
- net labels removed: RES2
- wire segments 462 -> 460
- no-connect marks 9 -> 16
Changed lines of the file:
@@
 Wire Wire Line
 	2000 1050 2100 1050
-Text Label 3850 1650 2    50   ~ 0
+Text Label 3850 1750 2    50   ~ 0
 RESET
-Wire Wire Line
-	3600 1650 3850 1650
 $Comp
 L 74xx:74HC74 URES1
@@
 	2500 950  2500 1050
 Connection ~ 2500 950
-Text Label 3850 1750 2    50   ~ 0
-RES2
 Wire Wire Line
 	3600 1750 3850 1750
-Text Label 8950 3950 0    50   ~ 0
-RES2
-Wire Wire Line
-	8950 3950 9200 3950
-Wire Wire Line
-	9200 3850 9200 3950
 Wire Wire Line
 	8700 3850 9100 3850
+NoConn ~ 3600 1650
+NoConn ~ 3600 1550
+NoConn ~ 3600 1450
+NoConn ~ 3600 1350
+NoConn ~ 3600 1250
+NoConn ~ 3600 1150
+NoConn ~ 3600 1000
+Wire Wire Line
+	9200 3850 9100 3850
+Connection ~ 9100 3850
 $EndSCHEMATC

Commit message: Get first test program to run
Parts:
- C3: value 100nF -> 10uF
- R3: value 1M -> 33k
Changed lines of the file:
@@
 P 750 900
 F 0 "C3" H 658 854 50  0000 R CNN
-F 1 "100nF" H 658 945 50  0000 R CNN
+F 1 "10uF" H 658 945 50  0000 R CNN
 F 2 "" H 750 900 50  0001 C CNN
 F 3 "~" H 750 900 50  0001 C CNN
@@
 P 750 1450
 F 0 "R3" H 809 1496 50  0000 L CNN
-F 1 "1M" H 809 1405 50  0000 L CNN
+F 1 "33k" H 809 1405 50  0000 L CNN
 F 2 "" H 750 1450 50  0001 C CNN
 F 3 "~" H 750 1450 50  0001 C CNN

Commit message: Design system breadboard Adjust emulator for new architecture
Parts:
- UIR1: value 74LS574 -> 74HC574
Changed lines of the file:
@@
 Text Label 5450 1150 1    50   ~ 0
 WR#
-Text Label 5550 1150 1    50   ~ 0
+Text Label 5650 1150 1    50   ~ 0
 RD#
 $Comp
@@
 L 74xx:74LS32 UOR1
 U 2 1 61E0D57E
-P 4900 1700
-F 0 "UOR1" H 4850 1900 50  0000 C CNN
-F 1 "74HC32" H 5100 1850 50  0000 C CNN
-F 2 "" H 4900 1700 50  0001 C CNN
-F 3 "http://www.ti.com/lit/gpn/sn74LS32" H 4900 1700 50  0001 C CNN
-	2    4900 1700
+P 4900 1250
+F 0 "UOR1" H 4850 1450 50  0000 C CNN
+F 1 "74HC32" H 5100 1400 50  0000 C CNN
+F 2 "" H 4900 1250 50  0001 C CNN
+F 3 "http://www.ti.com/lit/gpn/sn74LS32" H 4900 1250 50  0001 C CNN
+	2    4900 1250
 	1    0    0    -1
 $EndComp
@@
 Text Label 4250 900  0    50   ~ 0
 CMDOUT#
-Text Label 4300 1350 0    50   ~ 0
+Text Label 4300 1800 0    50   ~ 0
 CMDIN#
 Wire Wire Line
@@
 L 74xx:74LS32 UOR1
 U 4 1 644963BF
-P 4900 1250
-F 0 "UOR1" H 4850 1450 50  0000 C CNN
-F 1 "74HC32" H 5150 1400 50  0000 C CNN
-F 2 "" H 4900 1250 50  0001 C CNN
-F 3 "http://www.ti.com/lit/gpn/sn74LS32" H 4900 1250 50  0001 C CNN
-	4    4900 1250
+P 4900 1700
+F 0 "UOR1" H 4850 1900 50  0000 C CNN
+F 1 "74HC32" H 5150 1850 50  0000 C CNN
+F 2 "" H 4900 1700 50  0001 C CNN
+F 3 "http://www.ti.com/lit/gpn/sn74LS32" H 4900 1700 50  0001 C CNN
+	4    4900 1700
 	1    0    0    -1
 $EndComp
@@
 Wire Wire Line
 	5650 1700 5650 950
-Text Label 5650 1150 1    50   ~ 0
+Text Label 5550 1150 1    50   ~ 0
 WRX#
-Text Label 4300 1800 0    50   ~ 0
+Text Label 4300 1600 0    50   ~ 0
 CLK
 Wire Wire Line
@@
 Wire Wire Line
 	4250 900  4600 900
-Text Label 4300 1600 0    50   ~ 0
+Text Label 4300 1350 0    50   ~ 0
 CMDOP#
 Wire Wire Line
@@
 P 10400 2100
 F 0 "UIR1" V 10850 1550 50  0000 L CNN
-F 1 "74LS574" V 10750 1500 50  0000 L CNN
+F 1 "74HC574" V 10750 1500 50  0000 L CNN
 F 2 "" H 10400 2100 50  0001 C CNN
 F 3 "http://www.ti.com/lit/gpn/sn74LS574" H 10400 2100 50  0001 C CNN

Commit message: Fine-tune resistors of the oscillator
Parts:
- R1: value 22 -> 1k
- R2: value 220k -> 1M
Changed lines of the file:
@@
 P 1300 4000
 F 0 "R1" H 1359 4046 50  0000 L CNN
-F 1 "22" H 1359 3955 50  0000 L CNN
+F 1 "1k" H 1359 3955 50  0000 L CNN
 F 2 "" H 1300 4000 50  0001 C CNN
 F 3 "~" H 1300 4000 50  0001 C CNN
@@
 P 1000 3800
 F 0 "R2" V 804 3800 50  0000 C CNN
-F 1 "220k" V 895 3800 50  0000 C CNN
+F 1 "1M" V 895 3800 50  0000 C CNN
 F 2 "" H 1000 3800 50  0001 C CNN
 F 3 "~" H 1000 3800 50  0001 C CNN

Commit message: Change branch instruction to only use the B operator.
Parts:
- removed unit 3 of URES1
Connections:
- net labels added: CMDBBZ#
- net labels removed: CMDBEQ#
- wire segments 460 -> 470
Changed lines of the file:
@@
 CMDIN#
 Text Label 6800 2900 0    50   ~ 0
-CMDBEQ#
+CMDBBZ#
 Wire Wire Line
 	6800 2300 7200 2300
@@
 	3900 4100 3900 6550
 Wire Wire Line
-	3550 7250 3400 7250
+	3550 7250 3450 7250
 Connection ~ 3550 7250
 Wire Wire Line
-	3600 7150 3400 7150
+	3600 7150 3450 7150
 Connection ~ 3600 7150
 Wire Wire Line
-	3650 7050 3400 7050
+	3650 7050 3450 7050
 Connection ~ 3650 7050
 Wire Wire Line
-	3700 6950 3400 6950
+	3700 6950 3450 6950
 Connection ~ 3700 6950
 Wire Wire Line
@@
 $EndComp
 Text Label 3400 5450 2    50   ~ 0
-CMDBEQ#
+CMDBBZ#
 Wire Wire Line
 	3000 5450 3400 5450
@@
 Text Label 3850 1750 2    50   ~ 0
 RESET
-$Comp
-L 74xx:74HC74 URES1
-U 3 1 63A2E37D
-P 1550 7100
-F 0 "URES1" H 1650 7600 50  0000 L CNN
-F 1 "74HC74" H 1650 7500 50  0000 L CNN
-F 2 "" H 1550 7100 50  0001 C CNN
-F 3 "74xx/74hc_hct74.pdf" H 1550 7100 50  0001 C CNN
-	3    1550 7100
-	1    0    0    -1
-$EndComp
-$Comp
-L power:GND #PWR0142
-U 1 1 63A2E480
-P 1550 7550
-F 0 "#PWR0142" H 1550 7300 50  0001 C CNN
-F 1 "GND" H 1555 7377 50  0000 C CNN
-F 2 "" H 1550 7550 50  0001 C CNN
-F 3 "" H 1550 7550 50  0001 C CNN
-	1    1550 7550
-	1    0    0    -1
-$EndComp
-$Comp
-L power:+5V #PWR0143
-U 1 1 63A98EB3
-P 1550 6650
-F 0 "#PWR0143" H 1550 6500 50  0001 C CNN
-F 1 "+5V" H 1565 6823 50  0000 C CNN
-F 2 "" H 1550 6650 50  0001 C CNN
-F 3 "" H 1550 6650 50  0001 C CNN
-	1    1550 6650
-	1    0    0    -1
-$EndComp
-Wire Wire Line
-	1550 6650 1550 6700
-Wire Wire Line
-	1550 7550 1550 7500
 Text Label 9050 4050 0    50   ~ 0
 RESET
@@
 L Connector_Generic:Conn_01x08 JA1
 U 1 1 63E38A4B
-P 3200 6050
-F 0 "JA1" H 3200 5550 50  0000 C CNN
-F 1 "Conn_01x08" V 3300 6000 50  0000 C CNN
-F 2 "" H 3200 6050 50  0001 C CNN
-F 3 "~" H 3200 6050 50  0001 C CNN
-	1    3200 6050
+P 3250 6050
+F 0 "JA1" H 3250 5550 50  0000 C CNN
+F 1 "Conn_01x08" V 3350 6000 50  0000 C CNN
+F 2 "" H 3250 6050 50  0001 C CNN
+F 3 "~" H 3250 6050 50  0001 C CNN
+	1    3250 6050
 	-1   0    0    1
 $EndComp
@@
 L Connector_Generic:Conn_01x08 JB1
 U 1 1 63E38B1D
-P 3200 6950
-F 0 "JB1" H 3200 6450 50  0000 C CNN
-F 1 "Conn_01x08" V 3300 6950 50  0000 C CNN
-F 2 "" H 3200 6950 50  0001 C CNN
-F 3 "~" H 3200 6950 50  0001 C CNN
-	1    3200 6950
+P 3250 6950
+F 0 "JB1" H 3250 6450 50  0000 C CNN
+F 1 "Conn_01x08" V 3350 6950 50  0000 C CNN
+F 2 "" H 3250 6950 50  0001 C CNN
+F 3 "~" H 3250 6950 50  0001 C CNN
+	1    3250 6950
 	-1   0    0    1
 $EndComp
-Connection ~ 3400 7250
-Wire Wire Line
-	3400 7250 3000 7250
-Connection ~ 3400 7150
-Wire Wire Line
-	3400 7150 3000 7150
-Connection ~ 3400 7050
-Wire Wire Line
-	3400 7050 3000 7050
-Connection ~ 3400 6950
-Wire Wire Line
-	3400 6950 3000 6950
-Connection ~ 3400 6850
-Wire Wire Line
-	3400 6850 3000 6850
-Connection ~ 3400 6750
-Wire Wire Line
-	3400 6750 3000 6750
-Connection ~ 3400 6650
-Wire Wire Line
-	3400 6650 3000 6650
-Connection ~ 3400 6550
-Wire Wire Line
-	3400 6550 3000 6550
-Connection ~ 3400 6350
-Wire Wire Line
-	3400 6350 3000 6350
-Connection ~ 3400 6250
-Wire Wire Line
-	3400 6250 3000 6250
-Connection ~ 3400 6150
-Wire Wire Line
-	3400 6150 3000 6150
-Connection ~ 3400 6050
-Wire Wire Line
-	3400 6050 3000 6050
-Connection ~ 3400 5950
-Wire Wire Line
-	3400 5950 3000 5950
-Connection ~ 3400 5850
-Wire Wire Line
-	3400 5850 3000 5850
-Connection ~ 3400 5750
-Wire Wire Line
-	3400 5750 3000 5750
-Connection ~ 3400 5650
-Wire Wire Line
-	3400 5650 3000 5650
-Wire Wire Line
-	3400 5650 4000 5650
-Wire Wire Line
-	3400 5750 4050 5750
-Wire Wire Line
-	3400 5850 4100 5850
-Wire Wire Line
-	3400 5950 4150 5950
-Wire Wire Line
-	3400 6050 4200 6050
-Wire Wire Line
-	3400 6150 4250 6150
-Wire Wire Line
-	3400 6250 4300 6250
-Wire Wire Line
-	3400 6350 4350 6350
+Wire Wire Line
+	3450 5650 4000 5650
+Wire Wire Line
+	3450 5750 4050 5750
+Wire Wire Line
+	3450 5850 4100 5850
+Wire Wire Line
+	3450 5950 4150 5950
+Wire Wire Line
+	3450 6050 4200 6050
+Wire Wire Line
+	3450 6150 4250 6150
+Wire Wire Line
+	3450 6250 4300 6250
+Wire Wire Line
+	3450 6350 4350 6350
 $Comp
 L 74xx:74LS32 UOR1
@@
 	8450 1900 8450 1750
 $Comp
-L power:GND #PWR?
+L power:GND #PWR0138
 U 1 1 60B1A09C
 P 7400 1800
-F 0 "#PWR?" H 7400 1550 50  0001 C CNN
+F 0 "#PWR0138" H 7400 1550 50  0001 C CNN
 F 1 "GND" V 7405 1672 50  0000 R CNN
 F 2 "" H 7400 1800 50  0001 C CNN
@@
 	9050 800  9050 900
 $Comp
-L power:GND #PWR?
+L power:GND #PWR0139
 U 1 1 60E58593
 P 8050 1050
-F 0 "#PWR?" H 8050 800 50  0001 C CNN
+F 0 "#PWR0139" H 8050 800 50  0001 C CNN
 F 1 "GND" H 8055 877 50  0000 C CNN
 F 2 "" H 8050 1050 50  0001 C CNN
@@
 	5400 6650 5950 6650
 Wire Wire Line
-	3750 6550 3400 6550
-Wire Wire Line
-	3800 6650 3400 6650
-Wire Wire Line
-	3400 6850 3750 6850
-Wire Wire Line
-	3400 6750 3800 6750
-Wire Wire Line
-	3800 6650 3850 6650
-Wire Wire Line
-	3750 6550 3900 6550
+	3450 6850 3750 6850
+Wire Wire Line
+	3450 6750 3800 6750
 Wire Wire Line
 	9700 3850 9700 4400
@@
 	3800 6750 4400 6750
 Wire Wire Line
-	3800 4300 3800 6750
-Wire Wire Line
-	3750 4400 3750 6850
+	3800 4300 3800 6650
+Wire Wire Line
+	3750 4400 3750 6550
 $Comp
 L 74xx:74HC04 UCLK1
@@
 	2100 700  2500 700
 $Comp
-L power:+5V #PWR?
+L power:+5V #PWR0140
 U 1 1 60858F5C
 P 2450 950
-F 0 "#PWR?" H 2450 800 50  0001 C CNN
+F 0 "#PWR0140" H 2450 800 50  0001 C CNN
 F 1 "+5V" V 2465 1078 50  0000 L CNN
 F 2 "" H 2450 950 50  0001 C CNN
@@
 	9200 3850 9100 3850
 Connection ~ 9100 3850
+Connection ~ 3450 5650
+Connection ~ 3450 5750
+Connection ~ 3450 5850
+Connection ~ 3450 5950
+Connection ~ 3450 6050
+Connection ~ 3450 6150
+Connection ~ 3450 6250
+Connection ~ 3450 6350
+Wire Wire Line
+	3000 6350 3450 6350
+Wire Wire Line
+	3000 6250 3450 6250
+Wire Wire Line
+	3000 6150 3450 6150
+Wire Wire Line
+	3000 6050 3450 6050
+Wire Wire Line
+	3000 5950 3450 5950
+Wire Wire Line
+	3000 5850 3450 5850
+Wire Wire Line
+	3000 5750 3450 5750
+Wire Wire Line
+	3000 5650 3450 5650
+Wire Wire Line
+	3750 6550 3750 6850
+Wire Wire Line
+	3800 6650 3800 6750
+$Comp
+L power:GND #PWR0141
+U 1 1 60964FBC
+P 3050 7300
+F 0 "#PWR0141" H 3050 7050 50  0001 C CNN
+F 1 "GND" H 3055 7127 50  0000 C CNN
+F 2 "" H 3050 7300 50  0001 C CNN
+F 3 "" H 3050 7300 50  0001 C CNN
+	1    3050 7300
+	1    0    0    -1
+$EndComp
+Wire Wire Line
+	3050 7300 3050 7250
+Wire Wire Line
+	3050 6550 3000 6550
+Wire Wire Line
+	3000 6650 3050 6650
+Connection ~ 3050 6650
+Wire Wire Line
+	3050 6650 3050 6550
+Wire Wire Line
+	3000 6750 3050 6750
+Connection ~ 3050 6750
+Wire Wire Line
+	3050 6750 3050 6650
+Wire Wire Line
+	3000 6850 3050 6850
+Connection ~ 3050 6850
+Wire Wire Line
+	3050 6850 3050 6750
+Wire Wire Line
+	3000 6950 3050 6950
+Connection ~ 3050 6950
+Wire Wire Line
+	3050 6950 3050 6850
+Wire Wire Line
+	3000 7050 3050 7050
+Connection ~ 3050 7050
+Wire Wire Line
+	3050 7050 3050 6950
+Wire Wire Line
+	3000 7150 3050 7150
+Connection ~ 3050 7150
+Wire Wire Line
+	3050 7150 3050 7050
+Wire Wire Line
+	3000 7250 3050 7250
+Connection ~ 3050 7250
+Wire Wire Line
+	3050 7250 3050 7150
+$Comp
+L power:GND #PWR0142
+U 1 1 60B65DC9
+P 3300 550
+F 0 "#PWR0142" H 3300 300 50  0001 C CNN
+F 1 "GND" V 3305 422 50  0000 R CNN
+F 2 "" H 3300 550 50  0001 C CNN
+F 3 "" H 3300 550 50  0001 C CNN
+	1    3300 550
+	0    -1   -1   0
+$EndComp
+$Comp
+L power:+5V #PWR0143
+U 1 1 60B65EA6
+P 2800 550
+F 0 "#PWR0143" H 2800 400 50  0001 C CNN
+F 1 "+5V" V 2815 678 50  0000 L CNN
+F 2 "" H 2800 550 50  0001 C CNN
+F 3 "" H 2800 550 50  0001 C CNN
+	1    2800 550
+	0    -1   -1   0
+$EndComp
+Wire Wire Line
+	3300 550  3250 550
+Wire Wire Line
+	3250 550  3250 600
+Wire Wire Line
+	2800 550  3050 550
+Wire Wire Line
+	3050 550  3050 600
+Wire Wire Line
+	3450 6650 3850 6650
+Wire Wire Line
+	3450 6550 3900 6550
 $EndSCHEMATC

Commit message: Change address latch interface and software access. Refactor large parts of Bernd to work with new latch interface and make code more compact also.
Parts:
- removed JCTRL1: Conn_01x03, symbol Connector_Generic:Conn_01x03
- removed unit 2 of UOR1
- added J?: Conn_01x05, symbol Connector_Generic:Conn_01x05
Connections:
- net labels removed: WRX#
- wire segments 470 -> 469
Changed lines of the file:
@@
 	0    1    -1   0
 $EndComp
-Text Label 5450 1150 1    50   ~ 0
+Text Label 5250 1250 1    50   ~ 0
 WR#
-Text Label 5650 1150 1    50   ~ 0
+Text Label 5350 1250 1    50   ~ 0
 RD#
 $Comp
@@
 L 74xx:74LS32 UOR1
 U 1 1 61E0D517
-P 4900 800
-F 0 "UOR1" H 4850 1000 50  0000 C CNN
-F 1 "74HC32" H 5100 950 50  0000 C CNN
-F 2 "" H 4900 800 50  0001 C CNN
-F 3 "http://www.ti.com/lit/gpn/sn74LS32" H 4900 800 50  0001 C CNN
-	1    4900 800
-	1    0    0    -1
-$EndComp
-$Comp
-L 74xx:74LS32 UOR1
-U 2 1 61E0D57E
-P 4900 1250
-F 0 "UOR1" H 4850 1450 50  0000 C CNN
-F 1 "74HC32" H 5100 1400 50  0000 C CNN
-F 2 "" H 4900 1250 50  0001 C CNN
-F 3 "http://www.ti.com/lit/gpn/sn74LS32" H 4900 1250 50  0001 C CNN
-	2    4900 1250
-	1    0    0    -1
-$EndComp
-Wire Wire Line
-	5450 950  5450 1200
-Wire Wire Line
-	5550 950  5550 1250
-Text Label 4300 700  0    50   ~ 0
+P 4700 1050
+F 0 "UOR1" H 4650 1250 50  0000 C CNN
+F 1 "74HC32" H 4900 1200 50  0000 C CNN
+F 2 "" H 4700 1050 50  0001 C CNN
+F 3 "http://www.ti.com/lit/gpn/sn74LS32" H 4700 1050 50  0001 C CNN
+	1    4700 1050
+	1    0    0    -1
+$EndComp
+Wire Wire Line
+	5250 950  5250 1300
+Text Label 4100 950  0    50   ~ 0
 CLK
-Text Label 4300 1150 0    50   ~ 0
+Text Label 5650 1250 1    50   ~ 0
 CLK
-Wire Wire Line
-	4300 1150 4600 1150
-Text Label 4250 900  0    50   ~ 0
+Text Label 4050 1150 0    50   ~ 0
 CMDOUT#
-Text Label 4300 1800 0    50   ~ 0
+Text Label 4100 1650 0    50   ~ 0
 CMDIN#
-Wire Wire Line
-	4300 1350 4600 1350
 $Comp
 L 74xx:74LS32 UOR1
@@
 Wire Wire Line
 	3450 6350 4350 6350
-$Comp
-L 74xx:74LS32 UOR1
-U 4 1 644963BF
-P 4900 1700
-F 0 "UOR1" H 4850 1900 50  0000 C CNN
-F 1 "74HC32" H 5150 1850 50  0000 C CNN
-F 2 "" H 4900 1700 50  0001 C CNN
-F 3 "http://www.ti.com/lit/gpn/sn74LS32" H 4900 1700 50  0001 C CNN
-	4    4900 1700
-	1    0    0    -1
-$EndComp
 Wire Wire Line
 	6550 1950 6550 4800
@@
 Wire Wire Line
 	7200 4100 6150 4100
-$Comp
-L Connector_Generic:Conn_01x03 JCTRL1
-U 1 1 64911D58
-P 5550 750
-F 0 "JCTRL1" V 5750 850 50  0000 R CNN
-F 1 "Conn_01x03" V 5650 1000 50  0000 R CNN
-F 2 "" H 5550 750 50  0001 C CNN
-F 3 "~" H 5550 750 50  0001 C CNN
-	1    5550 750
-	0    1    -1   0
-$EndComp
-Wire Wire Line
-	5450 1200 5300 1200
-Wire Wire Line
-	5300 1200 5300 800
-Wire Wire Line
-	5300 800  5200 800
-Wire Wire Line
-	4300 700  4600 700
-Wire Wire Line
-	5200 1250 5550 1250
-Wire Wire Line
-	5200 1700 5650 1700
-Wire Wire Line
-	5650 1700 5650 950
-Text Label 5550 1150 1    50   ~ 0
-WRX#
-Text Label 4300 1600 0    50   ~ 0
+Wire Wire Line
+	5250 1300 5100 1300
+Wire Wire Line
+	5100 1300 5100 1050
+Wire Wire Line
+	5100 1050 5000 1050
+Wire Wire Line
+	4100 950  4400 950
+Wire Wire Line
+	5000 1550 5350 1550
+Text Label 4100 1450 0    50   ~ 0
 CLK
 Wire Wire Line
-	4300 1600 4600 1600
-Wire Wire Line
-	4250 900  4600 900
-Text Label 4300 1350 0    50   ~ 0
-CMDOP#
-Wire Wire Line
-	4300 1800 4600 1800
+	4100 1450 4400 1450
+Wire Wire Line
+	4050 1150 4400 1150
+Wire Wire Line
+	4100 1650 4400 1650
 Wire Wire Line
 	6850 3800 7200 3800
@@
 Wire Wire Line
 	3450 6550 3900 6550
+$Comp
+L 74xx:74LS32 UOR1
+U 4 1 644963BF
+P 4700 1550
+F 0 "UOR1" H 4650 1750 50  0000 C CNN
+F 1 "74HC32" H 4950 1700 50  0000 C CNN
+F 2 "" H 4700 1550 50  0001 C CNN
+F 3 "http://www.ti.com/lit/gpn/sn74LS32" H 4700 1550 50  0001 C CNN
+	4    4700 1550
+	1    0    0    -1
+$EndComp
+$Comp
+L Connector_Generic:Conn_01x05 J?
+U 1 1 60A33E07
+P 5450 750
+F 0 "J?" V 5416 462 50  0000 R CNN
+F 1 "Conn_01x05" V 5325 462 50  0000 R CNN
+F 2 "" H 5450 750 50  0001 C CNN
+F 3 "~" H 5450 750 50  0001 C CNN
+	1    5450 750
+	0    -1   -1   0
+$EndComp
+Wire Wire Line
+	5650 1250 5650 950
+Text Label 5450 1250 1    50   ~ 0
+CMDA#
+Text Label 5550 1250 1    50   ~ 0
+CMDB#
+Wire Wire Line
+	5350 950  5350 1550
+Wire Wire Line
+	5450 950  5450 1250
+Wire Wire Line
+	5550 950  5550 1250
 $EndSCHEMATC
