File: board/board.kicad_pcb (KiCad board)
At the start: 2 copper layers, 45 parts, among them Y1 Crystal

Commit message: Modify ALU so I can build it with parts that are actually available.
Parts:
- removed DRIVER1: 74HC541, Package_DIP:DIP-20_W7.62mm
- removed NAND1: 74HC10, Package_DIP:DIP-14_W7.62mm
- removed NOR1: 74HC27, Package_DIP:DIP-14_W7.62mm
- removed URES1: 74HC164, Package_DIP:DIP-14_W7.62mm
- removed UTIM1: NE555, Package_DIP:DIP-8_W7.62mm
- added AND3: 74AC11, Package_DIP:DIP-14_W7.62mm, F.Cu at (50.8, 73.7)
- added AND4: 74AC11, Package_DIP:DIP-14_W7.62mm, F.Cu at (53.3, 114.3)
- added GATE1: 74HC541, Package_DIP:DIP-20_W7.62mm, F.Cu at (274.3, 106.7)
- added RES1: 74HC164, Package_DIP:DIP-14_W7.62mm, F.Cu at (345.4, 154.9)
- added TIM1: NE555, Package_DIP:DIP-8_W7.62mm, F.Cu at (348.0, 195.6)
- ADD1, ADD2: value 74HC283 -> 74AC283
- AND1, AND2: value 74HC08 -> 74AC08
- LOGIC1, LOGIC2: value 74HC00 -> 74AC00
- MUX1, MUX2, MUX3, MUX4: value 74HC153 -> 74AC153
Connections:
- AND1 pad 10: Net-(AND1-Pad10) -> /BreadBinCPU/ALU/OP3
- AND1 pad 13: Net-(AND1-Pad10) -> /BreadBinCPU/ALU/OP3
- AND1 pad 2: Net-(AND1-Pad10) -> /BreadBinCPU/ALU/OP3
- AND1 pad 5: Net-(AND1-Pad10) -> /BreadBinCPU/ALU/OP3
- AND2 pad 10: Net-(AND2-Pad10) -> /BreadBinCPU/ALU/OP3
- AND2 pad 13: Net-(AND2-Pad10) -> /BreadBinCPU/ALU/OP3
- AND2 pad 2: Net-(AND2-Pad10) -> /BreadBinCPU/ALU/OP3
- AND2 pad 5: Net-(AND2-Pad10) -> /BreadBinCPU/ALU/OP3
- INV1 pad 1: /AD23 -> Net-(C2-Pad1)
- INV1 pad 10: Net-(INV1-Pad10) -> /ROMSEL#
- INV1 pad 11: Net-(INV1-Pad11) -> /AD23
- INV1 pad 12: Net-(INV1-Pad11) -> Net-(INV1-Pad12)
- INV1 pad 13: Net-(C2-Pad1) -> /AD22
- INV1 pad 2: /ROMSEL# -> Net-(INV1-Pad2)
- INV1 pad 3: /AD22 -> Net-(INV1-Pad2)
- INV1 pad 5: GND -> Net-(INV1-Pad4)
- INV1 pad 6: Net-(INV1-Pad6) -> /BreadBinCPU/CLK
- INV1 pad 8: /BreadBinCPU/CLK -> Net-(INV1-Pad8)
- INV1 pad 9: Net-(INV1-Pad10) -> Net-(INV1-Pad4)
- MCODE1 pad 1: +5V -> GND
- MCODE1 pad 30: +5V -> GND
- MUX1 pad 7: Net-(DRIVER1-Pad2) -> /BreadBinCPU/ALU/Q0
- MUX1 pad 9: Net-(DRIVER1-Pad3) -> /BreadBinCPU/ALU/Q1
- MUX2 pad 7: Net-(DRIVER1-Pad4) -> /BreadBinCPU/ALU/Q2
- MUX2 pad 9: Net-(DRIVER1-Pad5) -> /BreadBinCPU/ALU/Q3
- MUX3 pad 7: Net-(DRIVER1-Pad6) -> /BreadBinCPU/ALU/Q4
- MUX3 pad 9: Net-(DRIVER1-Pad7) -> /BreadBinCPU/ALU/Q5
- MUX4 pad 7: Net-(DRIVER1-Pad8) -> /BreadBinCPU/ALU/Q6
- MUX4 pad 9: Net-(DRIVER1-Pad9) -> /BreadBinCPU/ALU/Q7
- OP1 pad 14: /BreadBinCPU/PAR0 -> GND
- OP1 pad 15: /BreadBinCPU/ALU/OP0 -> Net-(OP1-Pad15)
- OP1 pad 16: /BreadBinCPU/ALU/OP1 -> Net-(OP1-Pad16)
- OP1 pad 17: /BreadBinCPU/PAR1 -> GND
- OP1 pad 18: /BreadBinCPU/PAR2 -> GND
- OP1 pad 19: /BreadBinCPU/ALU/OP2 -> Net-(OP1-Pad19)
- OP1 pad 2: Net-(OP1-Pad2) -> /BreadBinCPU/ALU/OP3
- OP1 pad 3: GND -> /BreadBinCPU/PAR3
- OP1 pad 4: GND -> /BreadBinCPU/PAR2
- OP1 pad 5: Net-(OP1-Pad5) -> /BreadBinCPU/ALU/OP2
- OP1 pad 6: Net-(OP1-Pad6) -> /BreadBinCPU/ALU/OP1
- OP1 pad 7: GND -> /BreadBinCPU/PAR1
- OP1 pad 8: GND -> /BreadBinCPU/PAR0
- OP1 pad 9: Net-(OP1-Pad9) -> /BreadBinCPU/ALU/OP0
- OR1 pad 10: /BreadBinCPU/CMD2 -> /AD0
- OR1 pad 4: /BreadBinCPU/CMDBRE# -> /BreadBinCPU/CMD2
- OR1 pad 5: /AD0 -> /BreadBinCPU/CMD1
- OR1 pad 6: /BreadBinCPU/BRA# -> Net-(OR1-Pad6)
- OR1 pad 8: Net-(OR1-Pad8) -> /BreadBinCPU/BRA#
- OR1 pad 9: /BreadBinCPU/CMD1 -> /BreadBinCPU/CMDBRE#
- OR2 pad 5: Net-(INV1-Pad4) -> Net-(INV1-Pad12)
- R1 pad 1: Net-(INV1-Pad11) -> Net-(INV1-Pad2)
- R2 pad 1: Net-(INV1-Pad11) -> Net-(INV1-Pad2)
- REG1 pad 1: GND -> /BreadBinCPU/PAR4
- REG1 pad 11: /D0 -> /D7
- REG1 pad 12: /D1 -> /D6
- REG1 pad 13: /D2 -> /D5
- REG1 pad 15: /D3 -> /D4
- REG1 pad 16: /D4 -> /D3
- REG1 pad 17: /D5 -> /D2
- REG1 pad 18: /D6 -> /D1
- REG1 pad 19: /D7 -> /D0
- REG1 pad 2: GND -> /BreadBinCPU/PAR3
- REG1 pad 21: /BreadBinCPU/PAR0 -> GND
- REG1 pad 23: /BreadBinCPU/PAR1 -> GND
- REG1 pad 24: /BreadBinCPU/PAR2 -> GND
- REG1 pad 25: /BreadBinCPU/PAR3 -> GND
- REG1 pad 26: /BreadBinCPU/PAR4 -> GND
- REG1 pad 27: Net-(OR1-Pad8) -> Net-(OR1-Pad6)
- REG1 pad 3: GND -> /BreadBinCPU/PAR2
- REG1 pad 4: GND -> /BreadBinCPU/PAR1
- REG1 pad 5: GND -> /BreadBinCPU/PAR0
