File: board/ALU.sch (KiCad schematic (older format))
At the start: 13 parts

Commit message: Modify schematic to better match breadboard possibilities.
Parts:
- removed DRIVER1: 74HC541, symbol 74xx:74HCT541
- ADD1, ADD2, MUX1, MUX2, MUX3, MUX4: footprint (none) -> Package_DIP:DIP-16_W7.62mm
- AND1, AND2, LOGIC1, LOGIC2, NAND1, NOR1: footprint (none) -> Package_DIP:DIP-14_W7.62mm
Connections:
- net labels removed: OE1#, OE2#
- wire segments 257 -> 242

Commit message: Modify ALU so I can build it with parts that are actually available.
Parts:
- removed NAND1: 74HC10, Package_DIP:DIP-14_W7.62mm, symbol 74xx:74LS10
- removed NOR1: 74HC27, Package_DIP:DIP-14_W7.62mm, symbol 74xx:74LS27
- added AND3, AND4: 74AC11, Package_DIP:DIP-14_W7.62mm, symbol 74xx:74LS11
- ADD1, ADD2: value 74HC283 -> 74AC283
- AND1, AND2: value 74HC08 -> 74AC08
- LOGIC1, LOGIC2: value 74HC00 -> 74AC00
- MUX1, MUX2, MUX3, MUX4: value 74HC153 -> 74AC153
Connections:
- net labels added: OP3
- wire segments 242 -> 249
- no-connect marks 0 -> 2
Other:
- note added: "ALU operation summary\n0000 B \n0001 ZERO \n0010 FF \n0011 ZERO \n0100 CRY B+1 if A=255, else B \n0101 TOP 1, if A=255 and B=255\n0110 FF \n0111 ZERO \n1000 ADD (A+B) mod 255\n1001 OVF 1, if A+B>255\n1010 NAND A NAND B\n1011 REV revert bit order of A\n1100 CRY1 A+B+1 if A=255, else A+B\n1101 OVF1 1, if A+B+1>255\n1110 NAND\n1111 REV\n"
- note removed: "ALU operation summary\n000 ADD (A+B) mod 255\n001 OVF 1, if A+B>255\n010 NAND A NAND B\n011 REV revert bit order of A\n100 CRY B+1 if A=255, else B \n101 TOP 1, if A=255 and B=255\n110 FF always 255\n111 ZERO always 0"

Commit message: Rework ALU to have 4 operand inputs and so it can be built with availbale parts
Parts:
- AND1, AND2: value 74AC08 -> 74HC08
- LOGIC1, LOGIC2: value 74AC00 -> 74HC00
Connections:
- wire segments 249 -> 250
Changed lines of the file:
@@
 	7350 650  9550 650
 Wire Wire Line
-	9550 650  9550 2150
-Wire Wire Line
 	8050 900  8050 800
 Wire Wire Line
 	8050 800  9450 800
 Wire Wire Line
-	9450 800  9450 2250
-Wire Wire Line
 	7350 2300 7350 2200
 Wire Wire Line
 	7350 2200 9350 2200
-Wire Wire Line
-	9350 2200 9350 2350
 Wire Wire Line
 	7350 3700 7350 3600
@@
 	8050 3700 9350 3700
 Wire Wire Line
-	9350 2650 9350 3700
-Wire Wire Line
 	7350 3600 9250 3600
 Wire Wire Line
-	9250 2550 9250 3600
-Wire Wire Line
 	7350 4950 9450 4950
-Wire Wire Line
-	9450 4950 9450 2750
 Wire Wire Line
 	8050 5050 9550 5050
@@
 P 5350 4200
 F 0 "LOGIC1" V 5350 4500 50  0000 R CNN
-F 1 "74AC00" V 5450 4500 50  0000 R CNN
+F 1 "74HC00" V 5450 4500 50  0000 R CNN
 F 2 "Package_DIP:DIP-14_W7.62mm" H 5350 4200 50  0001 C CNN
 F 3 "" H 5350 4200 50  0001 C CNN
@@
 P 5350 5550
 F 0 "LOGIC2" V 5350 5850 50  0000 R CNN
-F 1 "74AC00" V 5450 5850 50  0000 R CNN
+F 1 "74HC00" V 5450 5850 50  0000 R CNN
 F 2 "Package_DIP:DIP-14_W7.62mm" H 5350 5550 50  0001 C CNN
 F 3 "" H 5350 5550 50  0001 C CNN
@@
 	6200 3500 6200 3300
 Text Label 6050 3600 3    50   ~ 0
+NND3
+Text Label 5750 3600 3    50   ~ 0
+NND2
+Text Label 5950 4800 1    50   ~ 0
 NND0
-Text Label 5750 3600 3    50   ~ 0
+Text Label 5650 4800 1    50   ~ 0
 NND1
-Text Label 5950 4800 1    50   ~ 0
-NND2
-Text Label 5650 4800 1    50   ~ 0
-NND3
 Text Label 7350 2100 1    50   ~ 0
-ADD0
+ADD1
 Text Label 7550 2100 1    50   ~ 0
-NND0
+NND1
 Text Label 7450 2100 1    50   Italic 0
-OVF
+GND
 Text Label 7650 2100 1    50   Italic 0
-X7
+X6
 Wire Wire Line
 	7350 2100 7350 1900
@@
 	7650 2100 7650 1900
 Text Label 8050 2100 1    50   ~ 0
-ADD1
+ADD2
 Text Label 8250 2100 1    50   ~ 0
-NND1
+NND2
 Text Label 8150 2100 1    50   Italic 0
 GND
 Text Label 8350 2100 1    50   Italic 0
-X6
+X5
 Wire Wire Line
 	8050 2100 8050 1900
@@
 	8350 2100 8350 1900
 Text Label 7350 3500 1    50   ~ 0
-ADD2
+ADD0
 Text Label 7550 3500 1    50   ~ 0
-NND2
+NND0
 Text Label 7450 3500 1    50   Italic 0
 GND
 Text Label 7650 3500 1    50   Italic 0
-X5
+X7
 Wire Wire Line
 	7350 3500 7350 3300
@@
 	8350 3500 8350 3300
 Text Label 7350 4900 1    50   ~ 0
-ADD4
+ADD5
 Text Label 7550 4900 1    50   ~ 0
-NND4
+NND5
 Text Label 7450 4900 1    50   Italic 0
 GND
 Text Label 7650 4900 1    50   Italic 0
-X3
+X2
 Wire Wire Line
 	7350 4900 7350 4700
@@
 	7650 4900 7650 4700
 Text Label 8050 4900 1    50   ~ 0
-ADD5
+ADD6
 Text Label 8250 4900 1    50   ~ 0
-NND5
+NND6
 Text Label 8150 4900 1    50   Italic 0
 GND
 Text Label 8350 4900 1    50   Italic 0
-X2
+X1
 Wire Wire Line
 	8050 4900 8050 4700
@@
 	8350 4900 8350 4700
 Text Label 7350 6250 1    50   ~ 0
-ADD6
+ADD4
 Text Label 7550 6250 1    50   ~ 0
-NND6
+NND4
 Text Label 7450 6250 1    50   Italic 0
 GND
 Text Label 7650 6250 1    50   Italic 0
-X1
+X3
 Wire Wire Line
 	7350 6250 7350 6050
@@
 	5650 4800 5650 4550
 Text Label 6050 4950 3    50   Italic 0
+NND7
+Text Label 5750 4950 3    50   Italic 0
+NND6
+Text Label 5950 6150 1    50   Italic 0
 NND4
-Text Label 5750 4950 3    50   Italic 0
+Text Label 5650 6150 1    50   Italic 0
 NND5
-Text Label 5950 6150 1    50   Italic 0
-NND6
-Text Label 5650 6150 1    50   Italic 0
-NND7
 Wire Wire Line
 	5650 6150 5650 5900
@@
 	5500 2200 5500 2300
 Text Label 5950 3600 3    50   Italic 0
+X3
+Text Label 5850 3600 3    50   Italic 0
+B3
+Text Label 5650 3600 3    50   Italic 0
+X2
+Text Label 5550 3600 3    50   Italic 0
+B2
+Text Label 5850 4800 1    50   Italic 0
 X0
-Text Label 5850 3600 3    50   Italic 0
+Text Label 5750 4800 1    50   Italic 0
 B0
-Text Label 5650 3600 3    50   Italic 0
+Text Label 5550 4800 1    50   Italic 0
 X1
-Text Label 5550 3600 3    50   Italic 0
+Text Label 5450 4800 1    50   Italic 0
 B1
-Text Label 5850 4800 1    50   Italic 0
-X2
-Text Label 5750 4800 1    50   Italic 0
-B2
-Text Label 5550 4800 1    50   Italic 0
-X3
-Text Label 5450 4800 1    50   Italic 0
-B3
 Text Label 5950 4950 3    50   Italic 0
+X7
+Text Label 5850 4950 3    50   Italic 0
+B7
+Text Label 5650 4950 3    50   Italic 0
+X6
+Text Label 5550 4950 3    50   Italic 0
+B6
+Text Label 5850 6150 1    50   Italic 0
 X4
-Text Label 5850 4950 3    50   Italic 0
+Text Label 5750 6150 1    50   Italic 0
 B4
-Text Label 5650 4950 3    50   Italic 0
+Text Label 5550 6150 1    50   Italic 0
 X5
-Text Label 5550 4950 3    50   Italic 0
+Text Label 5450 6150 1    50   Italic 0
 B5
-Text Label 5850 6150 1    50   Italic 0
-X6
-Text Label 5750 6150 1    50   Italic 0
-B6
-Text Label 5550 6150 1    50   Italic 0
-X7
-Text Label 5450 6150 1    50   Italic 0
-B7
 Wire Wire Line
 	5850 6150 5850 5900
@@
 L 74xx:74LS08 AND1
 U 1 1 614EAA5B
+P 3800 2900
+F 0 "AND1" H 3800 3225 50  0000 C CNN
+F 1 "74HC08" H 3800 3134 50  0000 C CNN
+F 2 "Package_DIP:DIP-14_W7.62mm" H 3800 2900 50  0001 C CNN
+F 3 "http://www.ti.com/lit/gpn/sn74LS08" H 3800 2900 50  0001 C CNN
+	1    3800 2900
+	1    0    0    -1
+$EndComp
+$Comp
+L 74xx:74LS08 AND1
+U 2 1 614EAACC
 P 3800 2350
 F 0 "AND1" H 3800 2675 50  0000 C CNN
-F 1 "74AC08" H 3800 2584 50  0000 C CNN
+F 1 "74HC08" H 3800 2584 50  0000 C CNN
 F 2 "Package_DIP:DIP-14_W7.62mm" H 3800 2350 50  0001 C CNN
 F 3 "http://www.ti.com/lit/gpn/sn74LS08" H 3800 2350 50  0001 C CNN
-	1    3800 2350
-	1    0    0    -1
-$EndComp
-$Comp
-L 74xx:74LS08 AND1
-U 2 1 614EAACC
-P 3800 2900
-F 0 "AND1" H 3800 3225 50  0000 C CNN
-F 1 "74AC08" H 3800 3134 50  0000 C CNN
-F 2 "Package_DIP:DIP-14_W7.62mm" H 3800 2900 50  0001 C CNN
-F 3 "http://www.ti.com/lit/gpn/sn74LS08" H 3800 2900 50  0001 C CNN
-	2    3800 2900
+	2    3800 2350
 	1    0    0    -1
 $EndComp
@@
 L 74xx:74LS08 AND1
 U 3 1 614EAB33
+P 3800 4000
+F 0 "AND1" H 3800 4325 50  0000 C CNN
+F 1 "74HC08" H 3800 4234 50  0000 C CNN
+F 2 "Package_DIP:DIP-14_W7.62mm" H 3800 4000 50  0001 C CNN
+F 3 "http://www.ti.com/lit/gpn/sn74LS08" H 3800 4000 50  0001 C CNN
+	3    3800 4000
+	1    0    0    -1
+$EndComp
+$Comp
+L 74xx:74LS08 AND1
+U 4 1 614EAB90
 P 3800 3450
 F 0 "AND1" H 3800 3775 50  0000 C CNN
-F 1 "74AC08" H 3800 3684 50  0000 C CNN
+F 1 "74HC08" H 3800 3684 50  0000 C CNN
 F 2 "Package_DIP:DIP-14_W7.62mm" H 3800 3450 50  0001 C CNN
 F 3 "http://www.ti.com/lit/gpn/sn74LS08" H 3800 3450 50  0001 C CNN
-	3    3800 3450
-	1    0    0    -1
-$EndComp
-$Comp
-L 74xx:74LS08 AND1
-U 4 1 614EAB90
-P 3800 4000
-F 0 "AND1" H 3800 4325 50  0000 C CNN
-F 1 "74AC08" H 3800 4234 50  0000 C CNN
-F 2 "Package_DIP:DIP-14_W7.62mm" H 3800 4000 50  0001 C CNN
-F 3 "http://www.ti.com/lit/gpn/sn74LS08" H 3800 4000 50  0001 C CNN
-	4    3800 4000
+	4    3800 3450
 	1    0    0    -1
 $EndComp
@@
 P 6400 7000
 F 0 "AND1" H 6630 7046 50  0000 L CNN
-F 1 "74AC08" H 6630 6955 50  0000 L CNN
+F 1 "74HC08" H 6630 6955 50  0000 L CNN
 F 2 "Package_DIP:DIP-14_W7.62mm" H 6400 7000 50  0001 C CNN
 F 3 "http://www.ti.com/lit/gpn/sn74LS08" H 6400 7000 50  0001 C CNN
@@
 L 74xx:74LS08 AND2
 U 1 1 614EAC84
+P 3800 5100
+F 0 "AND2" H 3800 5425 50  0000 C CNN
+F 1 "74HC08" H 3800 5334 50  0000 C CNN
+F 2 "Package_DIP:DIP-14_W7.62mm" H 3800 5100 50  0001 C CNN
+F 3 "http://www.ti.com/lit/gpn/sn74LS08" H 3800 5100 50  0001 C CNN
+	1    3800 5100
+	1    0    0    -1
+$EndComp
+$Comp
+L 74xx:74LS08 AND2
+U 2 1 614EACF7
 P 3800 4550
 F 0 "AND2" H 3800 4875 50  0000 C CNN
-F 1 "74AC08" H 3800 4784 50  0000 C CNN
+F 1 "74HC08" H 3800 4784 50  0000 C CNN
 F 2 "Package_DIP:DIP-14_W7.62mm" H 3800 4550 50  0001 C CNN
 F 3 "http://www.ti.com/lit/gpn/sn74LS08" H 3800 4550 50  0001 C CNN
-	1    3800 4550
-	1    0    0    -1
-$EndComp
-$Comp
-L 74xx:74LS08 AND2
-U 2 1 614EACF7
-P 3800 5100
-F 0 "AND2" H 3800 5425 50  0000 C CNN
-F 1 "74AC08" H 3800 5334 50  0000 C CNN
-F 2 "Package_DIP:DIP-14_W7.62mm" H 3800 5100 50  0001 C CNN
-F 3 "http://www.ti.com/lit/gpn/sn74LS08" H 3800 5100 50  0001 C CNN
-	2    3800 5100
+	2    3800 4550
 	1    0    0    -1
 $EndComp
@@
 L 74xx:74LS08 AND2
 U 3 1 614EAD62
+P 3800 6200
+F 0 "AND2" H 3800 6525 50  0000 C CNN
+F 1 "74HC08" H 3800 6434 50  0000 C CNN
+F 2 "Package_DIP:DIP-14_W7.62mm" H 3800 6200 50  0001 C CNN
+F 3 "http://www.ti.com/lit/gpn/sn74LS08" H 3800 6200 50  0001 C CNN
+	3    3800 6200
+	1    0    0    -1
+$EndComp
+$Comp
+L 74xx:74LS08 AND2
+U 4 1 614EADCD
 P 3800 5650
 F 0 "AND2" H 3800 5975 50  0000 C CNN
-F 1 "74AC08" H 3800 5884 50  0000 C CNN
+F 1 "74HC08" H 3800 5884 50  0000 C CNN
 F 2 "Package_DIP:DIP-14_W7.62mm" H 3800 5650 50  0001 C CNN
 F 3 "http://www.ti.com/lit/gpn/sn74LS08" H 3800 5650 50  0001 C CNN
-	3    3800 5650
-	1    0    0    -1
-$EndComp
-$Comp
-L 74xx:74LS08 AND2
-U 4 1 614EADCD
-P 3800 6200
-F 0 "AND2" H 3800 6525 50  0000 C CNN
-F 1 "74AC08" H 3800 6434 50  0000 C CNN
-F 2 "Package_DIP:DIP-14_W7.62mm" H 3800 6200 50  0001 C CNN
-F 3 "http://www.ti.com/lit/gpn/sn74LS08" H 3800 6200 50  0001 C CNN
-	4    3800 6200
+	4    3800 5650
 	1    0    0    -1
 $EndComp
@@
 P 5650 7000
 F 0 "AND2" H 5880 7046 50  0000 L CNN
-F 1 "74AC08" H 5880 6955 50  0000 L CNN
+F 1 "74HC08" H 5880 6955 50  0000 L CNN
 F 2 "Package_DIP:DIP-14_W7.62mm" H 5650 7000 50  0001 C CNN
 F 3 "http://www.ti.com/lit/gpn/sn74LS08" H 5650 7000 50  0001 C CNN
@@
 	9450 2750 9900 2750
 Wire Wire Line
-	9350 2650 9900 2650
-Wire Wire Line
-	9250 2550 9900 2550
-Wire Wire Line
 	9250 2450 9900 2450
-Wire Wire Line
-	9350 2350 9900 2350
-Wire Wire Line
-	9450 2250 9900 2250
-Wire Wire Line
-	9550 2150 9900 2150
 $Comp
 L 74xx:74LS11 AND3
@@
 NoConn ~ 3700 7350
 NoConn ~ 2850 7350
+Wire Wire Line
+	9550 2250 9900 2250
+Wire Wire Line
+	9550 650  9550 2250
+Wire Wire Line
+	9450 800  9450 2350
+Wire Wire Line
+	9450 2350 9900 2350
+Wire Wire Line
+	9350 2200 9350 2150
+Wire Wire Line
+	9350 2150 9900 2150
+Wire Wire Line
+	9250 2650 9250 3600
+Wire Wire Line
+	9450 2750 9350 2750
+Wire Wire Line
+	9350 2750 9350 3700
+Wire Wire Line
+	9250 2650 9900 2650
+Wire Wire Line
+	9450 2550 9900 2550
+Wire Wire Line
+	9450 2550 9450 4950
 $EndSCHEMATC

Commit message: Modify ALU: Remove REV operation and get AVG/HALF/ROR instead.
Other:
- note added: "ALU operation summary\n0000 B B\n0001 ZERO always 0 \n0010 FF always 255 \n0011 HALF B/2 (rounded down) \n0100 CRY B+1 if A=255, else B \n0101 TOP 1, if A=255 and B=255\n0110 FF always 255\n0111 ?\n1000 ADD (A+B) mod 255\n1001 OVF 1, if A+B>255\n1010 NAND A NAND B\n1011 AVG (A+B)/2 (rounded down)\n1100 ?\n1101 ?\n1110 NAND\n1111 ROR \n"
- note removed: "ALU operation summary\n0000 B \n0001 ZERO \n0010 FF \n0011 ZERO \n0100 CRY B+1 if A=255, else B \n0101 TOP 1, if A=255 and B=255\n0110 FF \n0111 ZERO \n1000 ADD (A+B) mod 255\n1001 OVF 1, if A+B>255\n1010 NAND A NAND B\n1011 REV revert bit order of A\n1100 CRY1 A+B+1 if A=255, else A+B\n1101 OVF1 1, if A+B+1>255\n1110 NAND\n1111 REV\n"
Changed lines of the file:
@@
 GND
 Text Label 7650 2100 1    50   Italic 0
-X6
+ADD2
 Wire Wire Line
 	7350 2100 7350 1900
@@
 GND
 Text Label 8350 2100 1    50   Italic 0
-X5
+ADD3
 Wire Wire Line
 	8050 2100 8050 1900
@@
 NND0
 Text Label 7450 3500 1    50   Italic 0
-GND
+OVF
 Text Label 7650 3500 1    50   Italic 0
-X7
+ADD1
 Wire Wire Line
 	7350 3500 7350 3300
@@
 GND
 Text Label 8350 3500 1    50   Italic 0
-X4
+ADD4
 Wire Wire Line
 	8050 3500 8050 3300
@@
 GND
 Text Label 7650 4900 1    50   Italic 0
-X2
+ADD6
 Wire Wire Line
 	7350 4900 7350 4700
@@
 GND
 Text Label 8350 4900 1    50   Italic 0
-X1
+ADD7
 Wire Wire Line
 	8050 4900 8050 4700
@@
 GND
 Text Label 7650 6250 1    50   Italic 0
-X3
+ADD5
 Wire Wire Line
 	7350 6250 7350 6050
@@
 GND
 Text Label 8350 6250 1    50   Italic 0
-X0
+OVF
 Wire Wire Line
 	8050 6250 8050 6050
@@
 $EndComp
 Text Notes 9350 6500 0    50   ~ 0
-        ALU operation summary\n0000   B \n0001   ZERO        \n0010   FF              \n0011   ZERO                \n0100   CRY       B+1 if A=255, else B \n0101   TOP       1, if A=255 and B=255\n0110   FF          \n0111   ZERO    \n1000   ADD      (A+B) mod 255\n1001   OVF       1, if A+B>255\n1010   NAND     A NAND B\n1011   REV       revert bit order of A\n1100   CRY1    A+B+1  if A=255, else A+B\n1101   OVF1    1, if A+B+1>255\n1110   NAND\n1111   REV\n
+        ALU operation summary\n0000   B            B\n0001   ZERO     always 0   \n0010   FF           always 255   \n0011   HALF      B/2 (rounded down)         \n0100   CRY       B+1 if A=255, else B \n0101   TOP       1, if A=255 and B=255\n0110   FF           always 255\n0111                ?\n1000   ADD      (A+B) mod 255\n1001   OVF       1, if A+B>255\n1010   NAND     A NAND B\n1011   AVG       (A+B)/2  (rounded down)\n1100                ?\n1101                ?\n1110   NAND\n1111   ROR      \n
 $Comp
 L 74xx:74LS08 AND2

Commit message: Adjust schematics to match actual breadboard
Parts:
- renumbered AND3 to CMP1, AND4 to CMP2, LOGIC1 to NAND1, LOGIC2 to NAND2
Connections:
- wire segments 250 -> 257
Changed lines of the file:
@@
 $EndComp
 $Comp
-L Library:74HC00 LOGIC1
+L Library:74HC00 NAND1
 U 1 1 611AD906
 P 5350 4200
-F 0 "LOGIC1" V 5350 4500 50  0000 R CNN
+F 0 "NAND1" V 5350 4500 50  0000 R CNN
 F 1 "74HC00" V 5450 4500 50  0000 R CNN
 F 2 "Package_DIP:DIP-14_W7.62mm" H 5350 4200 50  0001 C CNN
@@
 $EndComp
 $Comp
-L Library:74HC00 LOGIC2
+L Library:74HC00 NAND2
 U 1 1 611AD9E1
 P 5350 5550
-F 0 "LOGIC2" V 5350 5850 50  0000 R CNN
+F 0 "NAND2" V 5350 5850 50  0000 R CNN
 F 1 "74HC00" V 5450 5850 50  0000 R CNN
 F 2 "Package_DIP:DIP-14_W7.62mm" H 5350 5550 50  0001 C CNN
@@
 	950  2250 2050 2250
 Wire Wire Line
-	950  2350 1950 2350
-Wire Wire Line
-	3100 2350 3100 2800
-Wire Wire Line
-	3100 2800 3500 2800
-Wire Wire Line
 	3350 6300 3350 5750
 Wire Wire Line
@@
 Wire Wire Line
 	3350 6300 3500 6300
-Wire Wire Line
-	3350 5750 3350 5200
-Wire Wire Line
-	3350 5200 3500 5200
 Connection ~ 3350 5750
 Wire Wire Line
-	3350 5200 3350 4650
-Wire Wire Line
-	3350 4650 3500 4650
-Connection ~ 3350 5200
-Wire Wire Line
 	3350 4100 3350 3550
 Wire Wire Line
@@
 Wire Wire Line
 	3350 4100 3500 4100
-Wire Wire Line
-	3350 3550 3350 3000
 Wire Wire Line
 	3350 3000 3500 3000
 Connection ~ 3350 3550
 Wire Wire Line
-	3350 3000 3350 2450
-Wire Wire Line
-	3350 2450 3500 2450
-Connection ~ 3350 3000
-Wire Wire Line
 	1050 6200 2200 6200
-Wire Wire Line
-	2200 2100 2300 2100
 Wire Wire Line
 	2900 2000 3250 2000
@@
 	2900 3900 3500 3900
 Wire Wire Line
-	950  2650 1650 2650
-Wire Wire Line
-	950  2750 1550 2750
-Wire Wire Line
-	950  2850 1450 2850
-Wire Wire Line
-	950  2950 1350 2950
-Wire Wire Line
-	3250 4550 3250 5000
-Wire Wire Line
-	3250 5000 3500 5000
-Wire Wire Line
-	3150 4650 3150 5550
-Wire Wire Line
-	3150 5550 3500 5550
-Wire Wire Line
-	3050 4750 3050 6100
-Wire Wire Line
-	3050 6100 3500 6100
-Wire Wire Line
-	1350 2950 1350 800
-Wire Wire Line
-	1350 800  2300 800
-Connection ~ 1350 2950
-Wire Wire Line
-	1450 2850 1450 900
-Wire Wire Line
-	1450 900  2300 900
-Connection ~ 1450 2850
-Wire Wire Line
-	1550 2750 1550 1000
-Wire Wire Line
-	1550 1000 2300 1000
-Connection ~ 1550 2750
-Wire Wire Line
-	1650 2650 1650 1350
-Wire Wire Line
-	1650 1350 2300 1350
-Connection ~ 1650 2650
+	2950 4650 2950 5550
+Wire Wire Line
+	2950 5550 3500 5550
+Wire Wire Line
+	2850 4750 2850 6100
+Wire Wire Line
+	2850 6100 3500 6100
 Wire Wire Line
 	1750 2550 1750 1450
@@
 	1850 2450 3000 2450
 Wire Wire Line
-	1950 2350 1950 1900
-Wire Wire Line
-	1950 1900 2300 1900
-Connection ~ 1950 2350
-Wire Wire Line
-	1950 2350 3100 2350
-Wire Wire Line
 	2050 2250 2050 2000
 Wire Wire Line
 	2050 2000 2300 2000
 Connection ~ 2050 2250
-Wire Wire Line
-	2050 2250 3500 2250
 Wire Wire Line
 	1050 6100 1500 6100
@@
 	9250 2450 9900 2450
 $Comp
-L 74xx:74LS11 AND3
+L 74xx:74LS11 CMP1
 U 1 1 60BAA425
-P 2600 900
-F 0 "AND3" H 2600 1225 50  0000 C CNN
-F 1 "74AC11" H 2600 1134 50  0000 C CNN
-F 2 "Package_DIP:DIP-14_W7.62mm" H 2600 900 50  0001 C CNN
-F 3 "http://www.ti.com/lit/gpn/sn74LS11" H 2600 900 50  0001 C CNN
-	1    2600 900
-	1    0    0    -1
-$EndComp
-$Comp
-L 74xx:74LS11 AND3
+P 3800 1450
+F 0 "CMP1" H 3800 1775 50  0000 C CNN
+F 1 "74AC11" H 3800 1684 50  0000 C CNN
+F 2 "Package_DIP:DIP-14_W7.62mm" H 3800 1450 50  0001 C CNN
+F 3 "http://www.ti.com/lit/gpn/sn74LS11" H 3800 1450 50  0001 C CNN
+	1    3800 1450
+	1    0    0    -1
+$EndComp
+$Comp
+L 74xx:74LS11 CMP1
 U 2 1 60BAA494
-P 2600 1450
-F 0 "AND3" H 2600 1775 50  0000 C CNN
-F 1 "74AC11" H 2600 1684 50  0000 C CNN
-F 2 "Package_DIP:DIP-14_W7.62mm" H 2600 1450 50  0001 C CNN
-F 3 "http://www.ti.com/lit/gpn/sn74LS11" H 2600 1450 50  0001 C CNN
-	2    2600 1450
-	1    0    0    -1
-$EndComp
-$Comp
-L 74xx:74LS11 AND3
+P 3400 7350
+F 0 "CMP1" H 3400 7675 50  0000 C CNN
+F 1 "74AC11" H 3400 7584 50  0000 C CNN
+F 2 "Package_DIP:DIP-14_W7.62mm" H 3400 7350 50  0001 C CNN
+F 3 "http://www.ti.com/lit/gpn/sn74LS11" H 3400 7350 50  0001 C CNN
+	2    3400 7350
+	1    0    0    -1
+$EndComp
+$Comp
+L 74xx:74LS11 CMP1
 U 3 1 60BAA4F9
 P 2600 2000
-F 0 "AND3" H 2600 2325 50  0000 C CNN
+F 0 "CMP1" H 2600 2325 50  0000 C CNN
 F 1 "74AC11" H 2600 2234 50  0000 C CNN
 F 2 "Package_DIP:DIP-14_W7.62mm" H 2600 2000 50  0001 C CNN
@@
 $EndComp
 $Comp
-L 74xx:74LS11 AND4
+L 74xx:74LS11 CMP2
 U 1 1 60BACC70
-P 3800 1450
-F 0 "AND4" H 3800 1775 50  0000 C CNN
-F 1 "74AC11" H 3800 1684 50  0000 C CNN
-F 2 "Package_DIP:DIP-14_W7.62mm" H 3800 1450 50  0001 C CNN
-F 3 "http://www.ti.com/lit/gpn/sn74LS11" H 3800 1450 50  0001 C CNN
-	1    3800 1450
+P 2600 900
+F 0 "CMP2" H 2600 1225 50  0000 C CNN
+F 1 "74AC11" H 2600 1134 50  0000 C CNN
+F 2 "Package_DIP:DIP-14_W7.62mm" H 2600 900 50  0001 C CNN
+F 3 "http://www.ti.com/lit/gpn/sn74LS11" H 2600 900 50  0001 C CNN
+	1    2600 900
 	1    0    0    -1
 $EndComp
@@
 $EndComp
 $Comp
-L 74xx:74LS11 AND4
+L 74xx:74LS11 CMP2
 U 2 1 60BAE2AD
 P 2550 7350
-F 0 "AND4" H 2550 7675 50  0000 C CNN
+F 0 "CMP2" H 2550 7675 50  0000 C CNN
 F 1 "74AC11" H 2550 7584 50  0000 C CNN
 F 2 "Package_DIP:DIP-14_W7.62mm" H 2550 7350 50  0001 C CNN
@@
 $EndComp
 $Comp
-L 74xx:74LS11 AND4
+L 74xx:74LS11 CMP2
 U 3 1 60BAE31E
-P 3400 7350
-F 0 "AND4" H 3400 7675 50  0000 C CNN
-F 1 "74AC11" H 3400 7584 50  0000 C CNN
-F 2 "Package_DIP:DIP-14_W7.62mm" H 3400 7350 50  0001 C CNN
-F 3 "http://www.ti.com/lit/gpn/sn74LS11" H 3400 7350 50  0001 C CNN
-	3    3400 7350
+P 2600 1450
+F 0 "CMP2" H 2600 1775 50  0000 C CNN
+F 1 "74AC11" H 2600 1684 50  0000 C CNN
+F 2 "Package_DIP:DIP-14_W7.62mm" H 2600 1450 50  0001 C CNN
+F 3 "http://www.ti.com/lit/gpn/sn74LS11" H 2600 1450 50  0001 C CNN
+	3    2600 1450
 	1    0    0    -1
 $EndComp
@@
 	1050 6300 3350 6300
 Wire Wire Line
-	2200 2100 2200 6200
-Wire Wire Line
-	3350 4650 3350 4100
-Connection ~ 3350 4650
+	3350 4650 3350 4450
 Connection ~ 3350 4100
 Wire Wire Line
-	1650 2650 2800 2650
-Wire Wire Line
 	2800 2650 2800 4450
 Wire Wire Line
-	2800 4450 3500 4450
-Wire Wire Line
-	1550 2750 2700 2750
+	2800 4450 3150 4450
 Wire Wire Line
 	2700 2750 2700 4550
 Wire Wire Line
-	2700 4550 3250 4550
-Wire Wire Line
-	1450 2850 2600 2850
+	2700 4550 3050 4550
 Wire Wire Line
 	2600 2850 2600 4650
 Wire Wire Line
-	2600 4650 3150 4650
-Wire Wire Line
-	1350 2950 2500 2950
+	2600 4650 2950 4650
 Wire Wire Line
 	2500 2950 2500 4750
 Wire Wire Line
-	2500 4750 3050 4750
+	2500 4750 2850 4750
 Text Label 1500 6300 2    50   ~ 0
 OP3
@@
 Wire Wire Line
 	9450 2550 9450 4950
+Wire Wire Line
+	3100 3000 3350 3000
+Wire Wire Line
+	3100 2350 3100 3000
+Wire Wire Line
+	3350 2800 3500 2800
+Connection ~ 3350 2800
+Wire Wire Line
+	3350 2800 3350 3550
+Wire Wire Line
+	3350 2250 3500 2250
+Wire Wire Line
+	3350 2250 3350 2800
+Wire Wire Line
+	3200 2250 3200 2450
+Wire Wire Line
+	3200 2450 3500 2450
+Wire Wire Line
+	3350 4650 3350 5000
+Wire Wire Line
+	3050 4550 3050 5200
+Wire Wire Line
+	3350 5000 3500 5000
+Connection ~ 3350 5000
+Wire Wire Line
+	3350 5000 3350 5200
+Wire Wire Line
+	3350 5200 3350 5750
+Wire Wire Line
+	3150 4650 3150 4450
+Wire Wire Line
+	3150 4650 3500 4650
+Wire Wire Line
+	3500 4450 3350 4450
+Connection ~ 3350 4450
+Wire Wire Line
+	3350 4450 3350 4100
+Wire Wire Line
+	3050 5200 3500 5200
+Wire Wire Line
+	2200 1900 2300 1900
+Wire Wire Line
+	2200 1900 2200 6200
+Wire Wire Line
+	2050 2250 3200 2250
+Wire Wire Line
+	950  2350 1950 2350
+Wire Wire Line
+	1950 2350 1950 2100
+Wire Wire Line
+	1950 2100 2300 2100
+Connection ~ 1950 2350
+Wire Wire Line
+	1950 2350 3100 2350
+Wire Wire Line
+	950  2850 1450 2850
+Wire Wire Line
+	950  2950 1350 2950
+Wire Wire Line
+	950  2750 1550 2750
+Wire Wire Line
+	950  2650 1650 2650
+Connection ~ 1650 2650
+Wire Wire Line
+	1650 2650 2800 2650
+Wire Wire Line
+	1650 900  2300 900
+Wire Wire Line
+	1650 900  1650 2650
+Wire Wire Line
+	1550 2750 1550 800
+Connection ~ 1550 2750
+Wire Wire Line
+	1550 2750 2700 2750
+Wire Wire Line
+	1550 800  2300 800
+Wire Wire Line
+	1450 2850 1450 1000
+Wire Wire Line
+	1450 1000 2300 1000
+Connection ~ 1450 2850
+Wire Wire Line
+	1450 2850 2600 2850
+Wire Wire Line
+	1350 2950 1350 1350
+Wire Wire Line
+	1350 1350 2300 1350
+Connection ~ 1350 2950
+Wire Wire Line
+	1350 2950 2500 2950
 $EndSCHEMATC
