File: board/CPU.sch (KiCad schematic (older format))
At the start: 13 parts

Commit message: Complete ALU design
Parts:
- removed UALU1: SST39SF040, symbol Memory_Flash:SST39SF040
Connections:
- wire segments 403 -> 402
Changed lines of the file:
@@
 $Descr A4 11693 8268
 encoding utf-8
-Sheet 2 2
+Sheet 2 3
 Title "CPU"
 Date ""
@@
 Text Label 5150 6250 2    50   ~ 0
 CLK
-Text Label 3700 5450 0    50   ~ 0
+Text Label 5300 5150 2    50   ~ 0
 CLK
-$Comp
-L power:+5V #PWR0118
-U 1 1 60ADF214
-P 3950 5150
-F 0 "#PWR0118" H 3950 5000 50  0001 C CNN
-F 1 "+5V" V 3965 5278 50  0000 L CNN
-F 2 "" H 3950 5150 50  0001 C CNN
-F 3 "" H 3950 5150 50  0001 C CNN
-	1    3950 5150
-	0    -1   -1   0
-$EndComp
-Wire Wire Line
-	4000 5150 3950 5150
 NoConn ~ 4000 6750
 NoConn ~ 4000 6850
@@
 	9550 6350 9550 6250
 Wire Wire Line
-	4000 5450 3700 5450
+	4900 5150 5300 5150
 NoConn ~ 4000 6950
 NoConn ~ 4000 7050
@@
 Wire Wire Line
 	5000 6250 5150 6250
-Text Label 3700 5350 0    50   ~ 0
+Text Label 5300 5050 2    50   ~ 0
 CMDSET#
 Wire Wire Line
-	4000 5350 3700 5350
+	4900 5050 5300 5050
 $Comp
 L 74xx:74LS32 UOR1
@@
 $EndComp
 NoConn ~ 6850 2800
-$Comp
-L Memory_Flash:SST39SF040 UALU?
-U 1 1 60ADF209
-P 4600 4350
-AR Path="/6064DD84/60ADF209" Ref="UALU?"  Part="1"
-AR Path="/60ADF209" Ref="UALU?"  Part="1"
-AR Path="/60ADE4F9/60ADF209" Ref="UALU1"  Part="1"
-F 0 "UALU1" H 4600 4550 50  0000 C CNN
-F 1 "SST39SF040" H 4700 4650 50  0000 C CNN
-F 2 "" H 4600 4650 50  0001 C CNN
-F 3 "http://ww1.microchip.com/downloads/en/DeviceDoc/25022B.pdf" H 4600 4650 50  0001 C CNN
-	1    4600 4350
-	1    0    0    -1
-$EndComp
 Wire Wire Line
 	6200 4800 6200 7350
@@
 	5600 4200 5600 7350
 Wire Wire Line
-	4000 6450 3600 6450
-Wire Wire Line
-	3600 4950 4000 4950
-Wire Wire Line
-	4000 6550 3550 6550
-Wire Wire Line
-	3550 4850 4000 4850
-Wire Wire Line
-	4000 6650 3500 6650
-Wire Wire Line
-	3500 4750 4000 4750
-Wire Wire Line
-	5200 3150 6200 3150
-Wire Wire Line
-	5200 3250 6100 3250
-Wire Wire Line
-	5200 3350 6000 3350
-Wire Wire Line
-	5200 3450 5900 3450
-Wire Wire Line
-	5200 3550 5800 3550
-Wire Wire Line
-	5200 3650 5700 3650
-Wire Wire Line
-	5200 3750 5600 3750
-Wire Wire Line
-	5200 3850 5500 3850
+	4000 6450 3850 6450
+Wire Wire Line
+	3850 5150 4000 5150
+Wire Wire Line
+	4000 6550 3750 6550
+Wire Wire Line
+	3750 5050 4000 5050
+Wire Wire Line
+	4000 6650 3650 6650
+Wire Wire Line
+	3650 4950 4000 4950
 Wire Wire Line
 	5700 4200 5700 4300
@@
 	5500 3850 5500 4100
 Wire Wire Line
-	3600 4950 3600 6450
-Wire Wire Line
-	3550 4850 3550 6550
-Wire Wire Line
-	3500 4750 3500 6650
+	3850 5150 3850 6450
+Wire Wire Line
+	3750 5050 3750 6550
+Wire Wire Line
+	3650 4950 3650 6650
 Wire Wire Line
 	750  3150 1400 3150
@@
 	2100 3850 4000 3850
 Wire Wire Line
-	3000 5200 3000 3950
-Wire Wire Line
-	3000 3950 4000 3950
+	3000 5200 3000 4050
+Wire Wire Line
+	3000 4050 4000 4050
 Wire Wire Line
 	1400 5200 3000 5200
@@
 	1500 5300 3050 5300
 Wire Wire Line
-	3050 5300 3050 4050
-Wire Wire Line
-	3050 4050 4000 4050
+	3050 5300 3050 4150
+Wire Wire Line
+	3050 4150 4000 4150
 Wire Wire Line
 	1600 5400 3100 5400
 Wire Wire Line
-	3100 5400 3100 4150
-Wire Wire Line
-	3100 4150 4000 4150
+	3100 5400 3100 4250
+Wire Wire Line
+	3100 4250 4000 4250
 Wire Wire Line
 	1700 5500 3150 5500
 Wire Wire Line
-	3150 5500 3150 4250
-Wire Wire Line
-	3150 4250 4000 4250
+	3150 5500 3150 4350
+Wire Wire Line
+	3150 4350 4000 4350
 Wire Wire Line
 	1800 5600 3200 5600
 Wire Wire Line
-	3200 5600 3200 4350
-Wire Wire Line
-	3200 4350 4000 4350
+	3200 5600 3200 4450
+Wire Wire Line
+	3200 4450 4000 4450
 Wire Wire Line
 	1900 5700 3250 5700
 Wire Wire Line
-	3250 5700 3250 4450
-Wire Wire Line
-	3250 4450 4000 4450
+	3250 5700 3250 4550
+Wire Wire Line
+	3250 4550 4000 4550
 Wire Wire Line
 	2000 5800 3300 5800
 Wire Wire Line
-	3300 5800 3300 4550
-Wire Wire Line
-	3300 4550 4000 4550
+	3300 5800 3300 4650
+Wire Wire Line
+	3300 4650 4000 4650
 Wire Wire Line
 	2100 5900 3350 5900
 Wire Wire Line
-	3350 5900 3350 4650
-Wire Wire Line
-	3350 4650 4000 4650
+	3350 5900 3350 4750
+Wire Wire Line
+	3350 4750 4000 4750
 Text HLabel 5500 7350 3    50   Input ~ 0
 D7
@@
 Wire Wire Line
 	8950 4050 8950 3850
-$Comp
-L power:GND #PWR0150
-U 1 1 60ADF4ED
-P 4600 3050
-F 0 "#PWR0150" H 4600 2800 50  0001 C CNN
-F 1 "GND" V 4605 2922 50  0000 R CNN
-F 2 "" H 4600 3050 50  0001 C CNN
-F 3 "" H 4600 3050 50  0001 C CNN
-	1    4600 3050
-	-1   0    0    1
-$EndComp
+$Sheet
+S 4000 3050 900  2200
+U 60B2B055
+F0 "ALU" 50
+F1 "ALU.sch" 50
+F2 "A0" I L 4000 3150 50
+F3 "A1" I L 4000 3250 50
+F4 "A2" I L 4000 3350 50
+F5 "A3" I L 4000 3450 50
+F6 "A4" I L 4000 3550 50
+F7 "A5" I L 4000 3650 50
+F8 "A6" I L 4000 3750 50
+F9 "A7" I L 4000 3850 50
+F10 "B0" I L 4000 4050 50
+F11 "B1" I L 4000 4150 50
+F12 "B2" I L 4000 4250 50
+F13 "B3" I L 4000 4350 50
+F14 "B4" I L 4000 4450 50
+F15 "B5" I L 4000 4550 50
+F16 "B6" I L 4000 4650 50
+F17 "B7" I L 4000 4750 50
+F18 "OP0" I L 4000 4950 50
+F19 "OP1" I L 4000 5050 50
+F20 "OP2" I L 4000 5150 50
+F21 "Q0" I R 4900 3150 50
+F22 "Q1" I R 4900 3250 50
+F23 "Q2" I R 4900 3350 50
+F24 "Q3" I R 4900 3450 50
+F25 "Q4" I R 4900 3550 50
+F26 "Q5" I R 4900 3650 50
+F27 "Q6" I R 4900 3750 50
+F28 "Q7" I R 4900 3850 50
+F29 "OE1#" I R 4900 5050 50
+F30 "OE2#" I R 4900 5150 50
+$EndSheet
+Wire Wire Line
+	4900 3150 6200 3150
+Wire Wire Line
+	4900 3250 6100 3250
+Wire Wire Line
+	4900 3350 6000 3350
+Wire Wire Line
+	4900 3450 5900 3450
+Wire Wire Line
+	4900 3550 5800 3550
+Wire Wire Line
+	4900 3650 5700 3650
+Wire Wire Line
+	4900 3750 5600 3750
+Wire Wire Line
+	4900 3850 5500 3850
 $EndSCHEMATC

Commit message: Modify schematic to better match breadboard possibilities.
Parts:
- added DRIVER?: 74HC541, Package_DIP:DIP-20_W7.62mm, symbol 74xx:74HCT541
- DEC1: renamed from UDEC1; footprint (none) -> Package_DIP:DIP-16_W7.62mm
- IR1: renamed from UIR1; footprint (none) -> Package_DIP:DIP-20_W7.62mm
- MCODE1: renamed from UCODE1; footprint (none) -> Package_DIP:DIP-32_W15.24mm
- OP1: renamed from UOP1; footprint (none) -> Package_DIP:DIP-20_W7.62mm
- OR1: renamed from UOR1; footprint (none) -> Package_DIP:DIP-14_W7.62mm
- PC1: renamed from UPC1; footprint (none) -> Package_DIP:DIP-16_W7.62mm
- PC2: renamed from UPC2; footprint (none) -> Package_DIP:DIP-16_W7.62mm
- PC3: renamed from UPC3; footprint (none) -> Package_DIP:DIP-20_W7.62mm
- REG1: renamed from UREG1; footprint (none) -> Package_DIP:DIP-28_W7.62mm
- UA1, UB1, UC1: footprint (none) -> Package_DIP:DIP-20_W7.62mm
Connections:
- wire segments 402 -> 409

Commit message: Modify ALU so I can build it with parts that are actually available.
Parts:
- gave numbers to parts that had none: 1
Connections:
- wire segments 409 -> 413
- no-connect marks 7 -> 6
Changed lines of the file:
@@
 Text Label 10550 1500 1    50   ~ 0
 PAR0
-Text Label 4950 6450 2    50   ~ 0
+Text Label 4950 6850 2    50   ~ 0
 PAR0
-Text Label 4950 6850 2    50   ~ 0
+Text Label 4950 6950 2    50   ~ 0
 PAR1
-Text Label 4950 6650 2    50   ~ 0
+Text Label 4950 7050 2    50   ~ 0
 PAR2
-Wire Wire Line
-	4750 6450 4950 6450
-Wire Wire Line
-	4750 6650 4950 6650
 Text Label 10250 6450 1    50   ~ 0
 PAR0
@@
 Wire Wire Line
 	9550 6350 9550 6250
-NoConn ~ 3750 6950
-NoConn ~ 3750 7050
-NoConn ~ 3750 7150
 Text Label 8150 6450 1    50   ~ 0
 BRA#
@@
 L 74xx:74LS32 OR1
 U 3 1 60ADF3D0
-P 8550 1950
-F 0 "OR1" H 8550 1600 50  0000 C CNN
-F 1 "74HC32" H 8550 1700 50  0000 C CNN
-F 2 "Package_DIP:DIP-14_W7.62mm" H 8550 1950 50  0001 C CNN
-F 3 "http://www.ti.com/lit/gpn/sn74LS32" H 8550 1950 50  0001 C CNN
-	3    8550 1950
-	-1   0    0    1
+P 3600 2800
+F 0 "OR1" H 3600 2450 50  0000 C CNN
+F 1 "74HC32" H 3600 2550 50  0000 C CNN
+F 2 "Package_DIP:DIP-14_W7.62mm" H 3600 2800 50  0001 C CNN
+F 3 "http://www.ti.com/lit/gpn/sn74LS32" H 3600 2800 50  0001 C CNN
+	3    3600 2800
+	1    0    0    -1
 $EndComp
 $Comp
@@
 	1    0    0    -1
 $EndComp
-Wire Wire Line
-	9150 2300 9150 1850
 Wire Wire Line
 	7200 1550 7200 1800
@@
 	9550 2050 9550 2000
 Wire Wire Line
-	9250 1400 9250 2050
-Wire Wire Line
-	9350 1500 9350 2500
+	9250 1400 9250 1850
+Wire Wire Line
+	9350 1500 9350 2050
 Wire Wire Line
 	2850 1750 2850 2550
@@
 L 74xx:74LS32 OR1
 U 2 1 62CEB51D
-P 3600 2800
-F 0 "OR1" H 4050 2950 50  0000 L CNN
-F 1 "74HC32" H 3700 2950 50  0000 L CNN
-F 2 "Package_DIP:DIP-14_W7.62mm" H 3600 2800 50  0001 C CNN
-F 3 "http://www.ti.com/lit/gpn/sn74LS32" H 3600 2800 50  0001 C CNN
-	2    3600 2800
-	1    0    0    -1
+P 8550 1950
+F 0 "OR1" H 8550 1650 50  0000 L CNN
+F 1 "74HC32" H 8500 1750 50  0000 L CNN
+F 2 "Package_DIP:DIP-14_W7.62mm" H 8550 1950 50  0001 C CNN
+F 3 "http://www.ti.com/lit/gpn/sn74LS32" H 8550 1950 50  0001 C CNN
+	2    8550 1950
+	-1   0    0    1
 $EndComp
 Text Label 4150 2800 2    50   ~ 0
@@
 	8950 4050 8950 3850
 $Sheet
-S 3650 3050 650  2200
+S 3650 3050 650  2300
 U 60B2B055
 F0 "ALU" 50
@@
 F27 "Q6" I R 4300 3750 50
 F28 "Q7" I R 4300 3850 50
+F29 "OP3" I L 3650 5250 50
 $EndSheet
 $Comp
@@
 Wire Wire Line
 	4750 6850 4950 6850
-Wire Wire Line
-	5000 6750 5000 6950
-Wire Wire Line
-	4750 6750 5000 6750
-Wire Wire Line
-	5000 6550 5000 6750
-Wire Wire Line
-	4750 6550 5000 6550
-Connection ~ 5000 6750
 $Comp
 L power:GND #PWR0138
 U 1 1 60ADF2EE
-P 5000 7200
-F 0 "#PWR0138" H 5000 6950 50  0001 C CNN
-F 1 "GND" H 5050 7050 50  0000 R CNN
-F 2 "" H 5000 7200 50  0001 C CNN
-F 3 "" H 5000 7200 50  0001 C CNN
-	1    5000 7200
+P 5200 6800
+F 0 "#PWR0138" H 5200 6550 50  0001 C CNN
+F 1 "GND" H 5250 6650 50  0000 R CNN
+F 2 "" H 5200 6800 50  0001 C CNN
+F 3 "" H 5200 6800 50  0001 C CNN
+	1    5200 6800
 	1    0    0    -1
 $EndComp
-Connection ~ 5000 6950
-Wire Wire Line
-	5000 6950 5000 7050
-Wire Wire Line
-	4750 6950 5000 6950
-Wire Wire Line
-	4750 7050 5000 7050
-Connection ~ 5000 7050
-Wire Wire Line
-	5000 7050 5000 7150
-Wire Wire Line
-	4750 7150 5000 7150
-Connection ~ 5000 7150
-Wire Wire Line
-	5000 7150 5000 7200
-NoConn ~ 3750 6550
 Wire Wire Line
 	3150 2900 3300 2900
@@
 P 4950 3650
 AR Path="/60ADE4F9/60B2B055/60C9A268" Ref="DRIVER?"  Part="1"
-AR Path="/60ADE4F9/60C9A268" Ref="DRIVER?"  Part="1"
-F 0 "DRIVER?" H 5200 4450 50  0000 C CNN
+AR Path="/60ADE4F9/60C9A268" Ref="GATE1"  Part="1"
+F 0 "GATE1" H 5200 4450 50  0000 C CNN
 F 1 "74HC541" H 5200 4350 50  0000 C CNN
 F 2 "Package_DIP:DIP-20_W7.62mm" H 4950 3650 50  0001 C CNN
@@
 P 4950 2800
 AR Path="/60ADE4F9/60B2B055/60C9A26F" Ref="#PWR?"  Part="1"
-AR Path="/60ADE4F9/60C9A26F" Ref="#PWR?"  Part="1"
-F 0 "#PWR?" H 4950 2650 50  0001 C CNN
+AR Path="/60ADE4F9/60C9A26F" Ref="#PWR0172"  Part="1"
+F 0 "#PWR0172" H 4950 2650 50  0001 C CNN
 F 1 "+5V" H 4965 2973 50  0000 C CNN
 F 2 "" H 4950 2800 50  0001 C CNN
@@
 P 4950 4500
 AR Path="/60ADE4F9/60B2B055/60C9A275" Ref="#PWR?"  Part="1"
-AR Path="/60ADE4F9/60C9A275" Ref="#PWR?"  Part="1"
-F 0 "#PWR?" H 4950 4250 50  0001 C CNN
+AR Path="/60ADE4F9/60C9A275" Ref="#PWR0173"  Part="1"
+F 0 "#PWR0173" H 4950 4250 50  0001 C CNN
 F 1 "GND" H 4955 4327 50  0000 C CNN
 F 2 "" H 4950 4500 50  0001 C CNN
@@
 	3650 4950 3450 4950
 Wire Wire Line
-	3450 4950 3450 6450
-Wire Wire Line
-	3450 6450 3750 6450
-Wire Wire Line
 	3650 5050 3500 5050
 Wire Wire Line
-	3500 5050 3500 6850
-Wire Wire Line
-	3500 6850 3750 6850
-Wire Wire Line
 	3650 5150 3550 5150
-Wire Wire Line
-	3550 5150 3550 6650
-Wire Wire Line
-	3550 6650 3750 6650
 Wire Wire Line
 	3150 3150 3650 3150
@@
 Wire Wire Line
 	8850 1850 9150 1850
-Connection ~ 9150 1850
-Wire Wire Line
-	9150 1850 9150 1300
-Wire Wire Line
-	8850 2050 9250 2050
-Connection ~ 9250 2050
 Wire Wire Line
 	9250 2050 9250 2400
@@
 Wire Wire Line
 	5800 1600 6700 1600
+Connection ~ 9350 2050
+Wire Wire Line
+	9350 2050 9350 2500
+Wire Wire Line
+	9150 1850 9250 1850
+Connection ~ 9250 1850
+Wire Wire Line
+	9250 1850 9250 2050
+Wire Wire Line
+	9150 1300 9150 2300
+Wire Wire Line
+	8850 2050 9350 2050
+Text Label 4950 7150 2    50   ~ 0
+PAR3
+Wire Wire Line
+	4950 6950 4750 6950
+Wire Wire Line
+	4750 7050 4950 7050
+Wire Wire Line
+	4950 7150 4750 7150
+Wire Wire Line
+	5200 6750 5200 6800
+Wire Wire Line
+	4750 6750 5200 6750
+Wire Wire Line
+	5200 6650 5200 6750
+Wire Wire Line
+	4750 6650 5200 6650
+Connection ~ 5200 6750
+Wire Wire Line
+	5200 6550 5200 6650
+Wire Wire Line
+	4750 6550 5200 6550
+Connection ~ 5200 6650
+Wire Wire Line
+	5200 6450 5200 6550
+Wire Wire Line
+	4750 6450 5200 6450
+Connection ~ 5200 6550
+Wire Wire Line
+	3650 5250 3600 5250
+Wire Wire Line
+	3600 5250 3600 7150
+Wire Wire Line
+	3600 7150 3750 7150
+Wire Wire Line
+	3750 7050 3550 7050
+Wire Wire Line
+	3550 5150 3550 7050
+Wire Wire Line
+	3750 6950 3500 6950
+Wire Wire Line
+	3500 5050 3500 6950
+Wire Wire Line
+	3750 6850 3450 6850
+Wire Wire Line
+	3450 4950 3450 6850
+NoConn ~ 3750 6650
+NoConn ~ 3750 6550
+NoConn ~ 3750 6450
 $EndSCHEMATC

Commit message: Rework ALU to have 4 operand inputs and so it can be built with availbale parts
Changed lines of the file:
@@
 Text Label 10550 1500 1    50   ~ 0
 PAR0
-Text Label 4950 6850 2    50   ~ 0
+Text Label 4950 7150 2    50   ~ 0
 PAR0
+Text Label 4950 7050 2    50   ~ 0
+PAR1
 Text Label 4950 6950 2    50   ~ 0
-PAR1
-Text Label 4950 7050 2    50   ~ 0
 PAR2
 Text Label 10250 6450 1    50   ~ 0
@@
 Wire Wire Line
 	8850 2050 9350 2050
-Text Label 4950 7150 2    50   ~ 0
+Text Label 4950 6850 2    50   ~ 0
 PAR3
 Wire Wire Line
@@
 Wire Wire Line
 	3650 5250 3600 5250
-Wire Wire Line
-	3600 5250 3600 7150
-Wire Wire Line
-	3600 7150 3750 7150
-Wire Wire Line
-	3750 7050 3550 7050
-Wire Wire Line
-	3550 5150 3550 7050
-Wire Wire Line
-	3750 6950 3500 6950
-Wire Wire Line
-	3500 5050 3500 6950
-Wire Wire Line
-	3750 6850 3450 6850
-Wire Wire Line
-	3450 4950 3450 6850
 NoConn ~ 3750 6650
 NoConn ~ 3750 6550
 NoConn ~ 3750 6450
+Wire Wire Line
+	3450 7150 3750 7150
+Wire Wire Line
+	3500 7050 3750 7050
+Wire Wire Line
+	3500 5050 3500 7050
+Wire Wire Line
+	3450 4950 3450 7150
+Wire Wire Line
+	3600 5250 3600 6850
+Wire Wire Line
+	3600 6850 3750 6850
+Wire Wire Line
+	3550 5150 3550 6950
+Wire Wire Line
+	3550 6950 3750 6950
 $EndSCHEMATC

Commit message: Work on ALU. Implement more 65c816 instructions.
Connections:
- net labels added: CMDNOP#
- wire segments 413 -> 414
- no-connect marks 6 -> 5
Changed lines of the file:
@@
 Text Label 4500 1800 1    50   ~ 0
 CMDOUT#
-Text Label 5100 1750 1    50   ~ 0
+Text Label 4900 1750 1    50   ~ 0
 CMDIN#
 $Comp
@@
 Wire Wire Line
 	4300 1750 4300 1450
-Text Label 4900 1750 1    50   ~ 0
+Text Label 5100 1750 1    50   ~ 0
 CLK
 Wire Wire Line
@@
 	0    -1   -1   0
 $EndComp
-NoConn ~ 6850 2800
 Wire Wire Line
 	6200 4800 6200 7350
@@
 Wire Wire Line
 	4750 6850 4950 6850
-$Comp
-L power:GND #PWR0138
-U 1 1 60ADF2EE
-P 5200 6800
-F 0 "#PWR0138" H 5200 6550 50  0001 C CNN
-F 1 "GND" H 5250 6650 50  0000 R CNN
-F 2 "" H 5200 6800 50  0001 C CNN
-F 3 "" H 5200 6800 50  0001 C CNN
-	1    5200 6800
-	1    0    0    -1
-$EndComp
 Wire Wire Line
 	3150 2900 3300 2900
@@
 	4950 7150 4750 7150
 Wire Wire Line
-	5200 6750 5200 6800
-Wire Wire Line
 	4750 6750 5200 6750
 Wire Wire Line
@@
 Wire Wire Line
 	4750 6650 5200 6650
-Connection ~ 5200 6750
 Wire Wire Line
 	5200 6550 5200 6650
@@
 Wire Wire Line
 	3550 6950 3750 6950
+Text Label 6450 2800 0    50   ~ 0
+CMDNOP#
+Wire Wire Line
+	6450 2800 6850 2800
+$Comp
+L power:+5V #PWR?
+U 1 1 60D0ACA7
+P 5200 6400
+F 0 "#PWR?" H 5200 6250 50  0001 C CNN
+F 1 "+5V" H 5215 6573 50  0000 C CNN
+F 2 "" H 5200 6400 50  0001 C CNN
+F 3 "" H 5200 6400 50  0001 C CNN
+	1    5200 6400
+	1    0    0    -1
+$EndComp
+Wire Wire Line
+	5200 6450 5200 6400
+Connection ~ 5200 6450
 $EndSCHEMATC

Commit message: Adjust schematics to match actual breadboard
Changed lines of the file:
@@
 Text Label 4900 6250 2    50   ~ 0
 CLK
-Text Label 5100 5000 2    50   ~ 0
+Text Label 5100 4900 2    50   ~ 0
 CLK
 NoConn ~ 3750 6750
@@
 Wire Wire Line
 	4750 6250 4900 6250
-Text Label 5100 4900 2    50   ~ 0
+Text Label 5100 5000 2    50   ~ 0
 CMDSET#
 $Comp
@@
 U 3 1 60ADF3D0
 P 3600 2800
-F 0 "OR1" H 3600 2450 50  0000 C CNN
-F 1 "74HC32" H 3600 2550 50  0000 C CNN
+F 0 "OR1" H 3350 2500 50  0000 C CNN
+F 1 "74HC32" H 3400 2600 50  0000 C CNN
 F 2 "Package_DIP:DIP-14_W7.62mm" H 3600 2800 50  0001 C CNN
 F 3 "http://www.ti.com/lit/gpn/sn74LS32" H 3600 2800 50  0001 C CNN

Commit message: Use a 1:2 clock duty cycle (33% low) no wait states are necessary
Connections:
- net labels added: CLKA, CLKB
- net labels removed: CLK
- wire segments 414 -> 415
- no-connect marks 5 -> 6
Changed lines of the file:
@@
 $EndComp
 Text Label 4900 6250 2    50   ~ 0
-CLK
+CLKA
 Text Label 5100 4900 2    50   ~ 0
-CLK
+CLKA
 NoConn ~ 3750 6750
 $Comp
@@
 $EndComp
 Text Label 7200 1800 1    50   ~ 0
-CLK
+CLKB
 $Comp
 L 74xx:74LS138 UDEC?
@@
 	9950 4950 9950 3850
 Text Label 6500 3900 0    50   ~ 0
-CLK
+CLKB
 Text Label 7850 6450 1    50   ~ 0
-CLK
+CLKB
 Wire Wire Line
 	7850 6250 7850 6450
 Text Label 9750 6450 1    50   ~ 0
-CLK
+CLKB
 Wire Wire Line
 	9750 6250 9750 6450
@@
 $EndComp
 Text Label 4300 1750 1    50   ~ 0
-CLK
+CLKA
 Text Label 4500 1800 1    50   ~ 0
 CMDOUT#
@@
 	4300 1750 4300 1450
 Text Label 5100 1750 1    50   ~ 0
-CLK
+CLKA
 Wire Wire Line
 	4900 1750 4900 1450
@@
 $EndComp
 Text Label 10750 2750 1    50   ~ 0
-CLK
+CLKB
 $Comp
 L power:GND #PWR0151
@@
 CMDX#
 Text Label 2300 5950 3    50   ~ 0
-CLK
+CLKA
 Connection ~ 1400 5200
 Connection ~ 1500 5300
@@
 CMDX#
 Text Label 2300 3900 3    50   ~ 0
-CLK
+CLKA
 Wire Wire Line
 	2300 4100 2300 3900
@@
 CMDX#
 Text Label 2300 1850 3    50   ~ 0
-CLK
+CLKA
 Wire Wire Line
 	2300 2050 2300 1850
@@
 	5000 850  5000 800
 Text HLabel 3750 800  1    50   Input ~ 0
-CLK
+CLKA
 Text HLabel 3950 800  1    50   Input ~ 0
 RES#
 Text Label 3750 1050 1    50   ~ 0
-CLK
+CLKA
 Text Label 3950 1050 1    50   ~ 0
 RES#
@@
 	6450 2800 6850 2800
 $Comp
-L power:+5V #PWR?
+L power:+5V #PWR0193
 U 1 1 60D0ACA7
 P 5200 6400
-F 0 "#PWR?" H 5200 6250 50  0001 C CNN
+F 0 "#PWR0193" H 5200 6250 50  0001 C CNN
 F 1 "+5V" H 5215 6573 50  0000 C CNN
 F 2 "" H 5200 6400 50  0001 C CNN
@@
 	5200 6450 5200 6400
 Connection ~ 5200 6450
+Text HLabel 3600 800  1    50   Input ~ 0
+CLKB
+Text Label 3600 1050 1    50   ~ 0
+CLKB
+Wire Wire Line
+	3600 1050 3600 800
+NoConn ~ 6450 2800
 $EndSCHEMATC

Commit message: Rework MMU to use a 74HC138 as in the OS816 reference
Connections:
- net labels added: CLKLATE, MEM#, RWB
- net labels removed: RD#, WR#
- wire segments 415 -> 419
- no-connect marks 6 -> 7
Changed lines of the file:
@@
 	1    0    0    1
 $EndComp
-Text Label 7200 1800 1    50   ~ 0
-CLKB
+Text Label 7200 1900 1    50   ~ 0
+CLKLATE
 $Comp
 L 74xx:74LS138 UDEC?
@@
 Text Label 6450 2600 0    50   ~ 0
 CMDOP#
+Text Label 6450 2400 0    50   ~ 0
+CMDSET#
 Text Label 6450 2300 0    50   ~ 0
-CMDSET#
-Text Label 6450 2400 0    50   ~ 0
 CMDIN#
 Text Label 6450 2900 0    50   ~ 0
@@
 L 74xx:74LS32 OR1
 U 1 1 60ADF3B1
-P 4400 1150
-F 0 "OR1" V 4700 950 50  0000 C CNN
-F 1 "74HC32" V 4600 950 50  0000 C CNN
-F 2 "Package_DIP:DIP-14_W7.62mm" H 4400 1150 50  0001 C CNN
-F 3 "http://www.ti.com/lit/gpn/sn74LS32" H 4400 1150 50  0001 C CNN
-	1    4400 1150
+P 5000 1150
+F 0 "OR1" V 5300 950 50  0000 C CNN
+F 1 "74HC32" V 5200 950 50  0000 C CNN
+F 2 "Package_DIP:DIP-14_W7.62mm" H 5000 1150 50  0001 C CNN
+F 3 "http://www.ti.com/lit/gpn/sn74LS32" H 5000 1150 50  0001 C CNN
+	1    5000 1150
 	0    -1   -1   0
 $EndComp
-Text Label 4300 1750 1    50   ~ 0
-CLKA
-Text Label 4500 1800 1    50   ~ 0
+Text Label 4450 1600 1    50   ~ 0
 CMDOUT#
 Text Label 4900 1750 1    50   ~ 0
-CMDIN#
+CMD0
 $Comp
 L 74xx:74LS32 OR1
@@
 Connection ~ 5900 4500
 Wire Wire Line
-	4300 1750 4300 1450
-Text Label 5100 1750 1    50   ~ 0
-CLKA
-Wire Wire Line
-	4900 1750 4900 1450
-Wire Wire Line
-	4500 1800 4500 1450
-Wire Wire Line
-	5100 1750 5100 1450
-Wire Wire Line
 	6500 3800 6850 3800
 Wire Wire Line
@@
 $EndComp
 Wire Wire Line
-	7200 1550 7200 1800
+	7200 1550 7200 1900
 $Comp
 L power:GND #PWR0154
@@
 L 74xx:74LS32 OR1
 U 4 1 60ADF64A
-P 5000 1150
-F 0 "OR1" V 5300 950 50  0000 C CNN
-F 1 "74HC32" V 5200 950 50  0000 C CNN
-F 2 "Package_DIP:DIP-14_W7.62mm" H 5000 1150 50  0001 C CNN
-F 3 "http://www.ti.com/lit/gpn/sn74LS32" H 5000 1150 50  0001 C CNN
-	4    5000 1150
-	0    -1   -1   0
+P 2200 750
+F 0 "OR1" H 2500 850 50  0000 C CNN
+F 1 "74HC32" H 2450 950 50  0000 C CNN
+F 2 "Package_DIP:DIP-14_W7.62mm" H 2200 750 50  0001 C CNN
+F 3 "http://www.ti.com/lit/gpn/sn74LS32" H 2200 750 50  0001 C CNN
+	4    2200 750
+	1    0    0    1
 $EndComp
 Wire Wire Line
@@
 Wire Wire Line
 	3200 1850 6200 1850
-Text HLabel 4400 800  1    50   Input ~ 0
-WR#
+Text HLabel 4450 800  1    50   Input ~ 0
+RWB
 Text HLabel 5000 800  1    50   Input ~ 0
-RD#
-Wire Wire Line
-	4400 850  4400 800
+MEM#
 Wire Wire Line
 	5000 850  5000 800
@@
 	3600 1050 3600 800
 NoConn ~ 6450 2800
+Text Label 5100 1750 1    50   ~ 0
+CMD2
+Wire Wire Line
+	4900 1450 4900 1750
+Wire Wire Line
+	5100 1750 5100 1450
+Wire Wire Line
+	4450 1600 4450 800
+Text Label 1600 750  0    50   ~ 0
+CLKA
+Wire Wire Line
+	1900 850  1850 850
+Wire Wire Line
+	1850 850  1850 750
+Wire Wire Line
+	1850 750  1600 750
+Wire Wire Line
+	1850 750  1850 650
+Wire Wire Line
+	1850 650  1900 650
+Connection ~ 1850 750
+Text Label 2850 750  2    50   ~ 0
+CLKLATE
+Wire Wire Line
+	2500 750  2850 750
+NoConn ~ 6450 2300
 $EndSCHEMATC
