File: board/board.sch (KiCad schematic (older format))
At the start: 20 parts, among them Y1 Crystal

Commit message: Modify schematic to better match breadboard possibilities.
Parts:
- added unit 3 of INV1
- C1, C2, C3: footprint (none) -> Capacitor_THT:C_Disc_D4.7mm_W2.5mm_P5.00mm
- C4: renamed from C10; footprint (none) -> Capacitor_THT:CP_Radial_D10.0mm_P5.00mm
- IN1: renamed from UIN1; footprint (none) -> Package_DIP:DIP-20_W7.62mm
- INV1: renamed from UINV1; footprint (none) -> Package_DIP:DIP-14_W7.62mm
- JIN1, JOUT1: footprint (none) -> Connector_PinHeader_2.54mm:PinHeader_1x08_P2.54mm_Vertical
- JPOWER1: footprint (none) -> Connector_PinHeader_2.54mm:PinHeader_1x02_P2.54mm_Vertical
- OR2: renamed from UOR2; footprint (none) -> Package_DIP:DIP-14_W7.62mm
- OUT1: renamed from UOUT1; footprint (none) -> Package_DIP:DIP-20_W7.62mm
- R1, R2, R3: footprint (none) -> Resistor_THT:R_Axial_DIN0204_L3.6mm_D1.6mm_P7.62mm_Horizontal
- RAM1: renamed from URAM1; footprint PDIP-32 -> Package_DIP:DIP-32_W15.24mm
- RES1: renamed from URES1; footprint (none) -> Package_DIP:DIP-14_W7.62mm
- ROM1: renamed from UROM1; footprint PDIP-32 -> Package_DIP:DIP-32_W15.24mm
- TIM1: renamed from UTIM1; footprint (none) -> Package_DIP:DIP-8_W7.62mm
- Y1: footprint (none) -> Crystal:Crystal_HC18-U_Vertical
Connections:
- net labels added: AD0, AD1, AD10, AD11, AD12, AD13, AD14, AD15, AD16, AD17, AD18, AD2, AD22, AD23, AD3, AD4, AD5, AD6, AD7, AD8, AD9
- net labels removed: A0, A1, A10, A11, A12, A13, A14, A15, A16, A17, A18, A2, A22, A23, A3, A4, A5, A6, A7, A8, A9
- wire segments 236 -> 237
- no-connect marks 13 -> 14
Other:
- moved on the sheet: INV1A, INV1B, INV1D, INV1E, INV1F

Commit message: Modify ALU so I can build it with parts that are actually available.
Parts:
- INV1: footprint (none) -> Package_DIP:DIP-14_W7.62mm
Changed lines of the file:
@@
 F 0 "INV1" H 2500 3817 50  0000 C CNN
 F 1 "74HC04" H 2500 3726 50  0000 C CNN
-F 2 "" H 2500 3500 50  0001 C CNN
+F 2 "Package_DIP:DIP-14_W7.62mm" H 2500 3500 50  0001 C CNN
 F 3 "http://www.nxp.com/documents/data_sheet/74HC_HCT04.pdf" H 2500 3500 50  0001 C CNN
 	3    2500 3500

Commit message: Adjust schematics to match actual breadboard
Parts:
- renumbered OR2 to MMU1
Changed lines of the file:
@@
 $EndComp
 $Comp
-L 74xx:74LS32 OR2
+L 74xx:74LS32 MMU1
 U 5 1 62016085
 P 6500 6900
-F 0 "OR2" H 6550 7400 50  0000 L CNN
+F 0 "MMU1" H 6550 7400 50  0000 L CNN
 F 1 "74HC32" H 6550 7300 50  0000 L CNN
 F 2 "Package_DIP:DIP-14_W7.62mm" H 6500 6900 50  0001 C CNN
@@
 Wire Wire Line
 	7300 4350 7300 4150
-Text Label 9800 5750 1    50   ~ 0
+Text Label 9600 5750 1    50   ~ 0
 D2
 Text Label 9700 5750 1    50   ~ 0
 D1
-Text Label 9600 5750 1    50   ~ 0
+Text Label 9800 5750 1    50   ~ 0
 D0
 Text Label 9500 5750 1    50   ~ 0
@@
 Wire Wire Line
 	8400 5750 8400 5550
-Text Label 9900 4150 3    50   ~ 0
+Text Label 9500 4150 3    50   ~ 0
 D3
-Text Label 9800 4150 3    50   ~ 0
+Text Label 9600 4150 3    50   ~ 0
 D4
 Text Label 9700 4150 3    50   ~ 0
 D5
-Text Label 9600 4150 3    50   ~ 0
+Text Label 9800 4150 3    50   ~ 0
 D6
-Text Label 9500 4150 3    50   ~ 0
+Text Label 9900 4150 3    50   ~ 0
 D7
 Text Label 9300 4150 3    50   ~ 0
@@
 AD22
 $Comp
-L 74xx:74LS32 OR2
+L 74xx:74LS32 MMU1
 U 1 1 60D820F3
 P 6750 2950
-F 0 "OR2" H 6750 3275 50  0000 C CNN
-F 1 "74HC32" H 6750 3184 50  0000 C CNN
+F 0 "MMU1" V 6650 2600 50  0000 C CNN
+F 1 "74HC32" V 6750 2600 50  0000 C CNN
 F 2 "Package_DIP:DIP-14_W7.62mm" H 6750 2950 50  0001 C CNN
 F 3 "http://www.ti.com/lit/gpn/sn74LS32" H 6750 2950 50  0001 C CNN
@@
 $EndComp
 $Comp
-L 74xx:74LS32 OR2
+L 74xx:74LS32 MMU1
 U 2 1 60D8215E
 P 9150 2950
-F 0 "OR2" H 9150 3275 50  0000 C CNN
-F 1 "74HC32" H 9150 3184 50  0000 C CNN
+F 0 "MMU1" V 9050 2600 50  0000 C CNN
+F 1 "74HC32" V 9150 2600 50  0000 C CNN
 F 2 "Package_DIP:DIP-14_W7.62mm" H 9150 2950 50  0001 C CNN
 F 3 "http://www.ti.com/lit/gpn/sn74LS32" H 9150 2950 50  0001 C CNN
@@
 $EndComp
 $Comp
-L 74xx:74LS32 OR2
+L 74xx:74LS32 MMU1
 U 3 1 60E5121A
 P 3350 6250
-F 0 "OR2" V 3396 6070 50  0000 R CNN
-F 1 "74HC32" V 3305 6070 50  0000 R CNN
+F 0 "MMU1" H 3750 6050 50  0000 R CNN
+F 1 "74HC32" H 3800 6150 50  0000 R CNN
 F 2 "Package_DIP:DIP-14_W7.62mm" H 3350 6250 50  0001 C CNN
 F 3 "http://www.ti.com/lit/gpn/sn74LS32" H 3350 6250 50  0001 C CNN
@@
 $EndComp
 $Comp
-L 74xx:74LS32 OR2
+L 74xx:74LS32 MMU1
 U 4 1 60F8B8F9
 P 3350 6800
-F 0 "OR2" V 3396 6620 50  0000 R CNN
-F 1 "74HC32" V 3305 6620 50  0000 R CNN
+F 0 "MMU1" H 3750 6600 50  0000 R CNN
+F 1 "74HC32" H 3800 6700 50  0000 R CNN
 F 2 "Package_DIP:DIP-14_W7.62mm" H 3350 6800 50  0001 C CNN
 F 3 "http://www.ti.com/lit/gpn/sn74LS32" H 3350 6800 50  0001 C CNN

Commit message: Use a 1:2 clock duty cycle (33% low) no wait states are necessary
Parts:
- added RV1: 1k, symbol Device:R_POT
- R3: value 33k -> 22k
Connections:
- wire segments 237 -> 244
- no-connect marks 14 -> 13
Other:
- moved on the sheet: INV1A
Changed lines of the file:
@@
 L Device:Crystal Y1
 U 1 1 62609387
-P 1650 3650
-F 0 "Y1" H 1650 3918 50  0000 C CNN
-F 1 "Crystal" H 1650 3827 50  0000 C CNN
-F 2 "Crystal:Crystal_HC18-U_Vertical" H 1650 3650 50  0001 C CNN
-F 3 "~" H 1650 3650 50  0001 C CNN
-	1    1650 3650
+P 1250 3650
+F 0 "Y1" H 1250 3918 50  0000 C CNN
+F 1 "Crystal" H 1250 3827 50  0000 C CNN
+F 2 "Crystal:Crystal_HC18-U_Vertical" H 1250 3650 50  0001 C CNN
+F 3 "~" H 1250 3650 50  0001 C CNN
+	1    1250 3650
 	1    0    0    -1
 $EndComp
@@
 L Device:C_Small C2
 U 1 1 62609613
-P 1350 3850
-F 0 "C2" H 1442 3896 50  0000 L CNN
-F 1 "33pF" H 1442 3805 50  0000 L CNN
-F 2 "Capacitor_THT:C_Disc_D4.7mm_W2.5mm_P5.00mm" H 1350 3850 50  0001 C CNN
-F 3 "~" H 1350 3850 50  0001 C CNN
-	1    1350 3850
+P 950 3850
+F 0 "C2" H 1042 3896 50  0000 L CNN
+F 1 "33pF" H 1042 3805 50  0000 L CNN
+F 2 "Capacitor_THT:C_Disc_D4.7mm_W2.5mm_P5.00mm" H 950 3850 50  0001 C CNN
+F 3 "~" H 950 3850 50  0001 C CNN
+	1    950  3850
 	1    0    0    -1
 $EndComp
@@
 L Device:C_Small C1
 U 1 1 6260970F
-P 1950 3850
-F 0 "C1" H 1750 3900 50  0000 L CNN
-F 1 "33pF" H 1700 3800 50  0000 L CNN
-F 2 "Capacitor_THT:C_Disc_D4.7mm_W2.5mm_P5.00mm" H 1950 3850 50  0001 C CNN
-F 3 "~" H 1950 3850 50  0001 C CNN
-	1    1950 3850
+P 1550 3850
+F 0 "C1" H 1350 3900 50  0000 L CNN
+F 1 "33pF" H 1300 3800 50  0000 L CNN
+F 2 "Capacitor_THT:C_Disc_D4.7mm_W2.5mm_P5.00mm" H 1550 3850 50  0001 C CNN
+F 3 "~" H 1550 3850 50  0001 C CNN
+	1    1550 3850
 	1    0    0    -1
 $EndComp
@@
 L power:GND #PWR0132
 U 1 1 62634084
-P 1350 4000
-F 0 "#PWR0132" H 1350 3750 50  0001 C CNN
-F 1 "GND" H 1355 3827 50  0000 C CNN
-F 2 "" H 1350 4000 50  0001 C CNN
-F 3 "" H 1350 4000 50  0001 C CNN
-	1    1350 4000
+P 950 4000
+F 0 "#PWR0132" H 950 3750 50  0001 C CNN
+F 1 "GND" H 955 3827 50  0000 C CNN
+F 2 "" H 950 4000 50  0001 C CNN
+F 3 "" H 950 4000 50  0001 C CNN
+	1    950  4000
 	1    0    0    -1
 $EndComp
@@
 L power:GND #PWR0133
 U 1 1 626340D0
-P 1950 4000
-F 0 "#PWR0133" H 1950 3750 50  0001 C CNN
-F 1 "GND" H 1955 3827 50  0000 C CNN
-F 2 "" H 1950 4000 50  0001 C CNN
-F 3 "" H 1950 4000 50  0001 C CNN
-	1    1950 4000
+P 1550 4000
+F 0 "#PWR0133" H 1550 3750 50  0001 C CNN
+F 1 "GND" H 1555 3827 50  0000 C CNN
+F 2 "" H 1550 4000 50  0001 C CNN
+F 3 "" H 1550 4000 50  0001 C CNN
+	1    1550 4000
 	1    0    0    -1
 $EndComp
@@
 L Device:R_Small R1
 U 1 1 62634131
-P 1950 3450
-F 0 "R1" H 2009 3496 50  0000 L CNN
-F 1 "1k" H 2009 3405 50  0000 L CNN
-F 2 "Resistor_THT:R_Axial_DIN0204_L3.6mm_D1.6mm_P7.62mm_Horizontal" H 1950 3450 50  0001 C CNN
-F 3 "~" H 1950 3450 50  0001 C CNN
-	1    1950 3450
+P 1550 3450
+F 0 "R1" H 1609 3496 50  0000 L CNN
+F 1 "1k" H 1609 3405 50  0000 L CNN
+F 2 "Resistor_THT:R_Axial_DIN0204_L3.6mm_D1.6mm_P7.62mm_Horizontal" H 1550 3450 50  0001 C CNN
+F 3 "~" H 1550 3450 50  0001 C CNN
+	1    1550 3450
 	1    0    0    -1
 $EndComp
@@
 L Device:R_Small R2
 U 1 1 626341D7
-P 1650 3250
-F 0 "R2" V 1454 3250 50  0000 C CNN
-F 1 "1M" V 1545 3250 50  0000 C CNN
-F 2 "Resistor_THT:R_Axial_DIN0204_L3.6mm_D1.6mm_P7.62mm_Horizontal" H 1650 3250 50  0001 C CNN
-F 3 "~" H 1650 3250 50  0001 C CNN
-	1    1650 3250
+P 1250 3250
+F 0 "R2" V 1054 3250 50  0000 C CNN
+F 1 "1M" V 1145 3250 50  0000 C CNN
+F 2 "Resistor_THT:R_Axial_DIN0204_L3.6mm_D1.6mm_P7.62mm_Horizontal" H 1250 3250 50  0001 C CNN
+F 3 "~" H 1250 3250 50  0001 C CNN
+	1    1250 3250
 	0    1    1    0
 $EndComp
 Wire Wire Line
-	1350 3750 1350 3650
-Wire Wire Line
-	1550 3250 1350 3250
-Connection ~ 1350 3250
-Wire Wire Line
-	1350 3250 1350 2850
-Connection ~ 1350 3650
-Wire Wire Line
-	1350 3650 1350 3250
+	950  3750 950  3650
+Wire Wire Line
+	1150 3250 950  3250
+Connection ~ 950  3250
+Wire Wire Line
+	950  3250 950  2850
+Connection ~ 950  3650
+Wire Wire Line
+	950  3650 950  3250
 $Comp
 L 74xx:74HC04 INV1
@@
 	5800 7400 5800 7450
 Wire Wire Line
-	1350 3650 1500 3650
-Wire Wire Line
-	1800 3650 1950 3650
-Wire Wire Line
-	1950 3650 1950 3750
-Wire Wire Line
-	1950 3650 1950 3550
-Connection ~ 1950 3650
-Wire Wire Line
-	1750 3250 1950 3250
-Connection ~ 1950 3250
-Wire Wire Line
-	1950 3250 1950 3350
-Wire Wire Line
-	1350 3950 1350 4000
-Wire Wire Line
-	1950 3950 1950 4000
+	950  3650 1100 3650
+Wire Wire Line
+	1400 3650 1550 3650
+Wire Wire Line
+	1550 3650 1550 3750
+Wire Wire Line
+	1550 3650 1550 3550
+Connection ~ 1550 3650
+Wire Wire Line
+	1350 3250 1550 3250
+Connection ~ 1550 3250
+Wire Wire Line
+	1550 3250 1550 3350
+Wire Wire Line
+	950  3950 950  4000
+Wire Wire Line
+	1550 3950 1550 4000
 $Comp
 L Timer:NE555 TIM1
@@
 P 1450 1800
 F 0 "R3" H 1509 1846 50  0000 L CNN
-F 1 "33k" H 1509 1755 50  0000 L CNN
+F 1 "22k" H 1509 1755 50  0000 L CNN
 F 2 "Resistor_THT:R_Axial_DIN0204_L3.6mm_D1.6mm_P7.62mm_Horizontal" H 1450 1800 50  0001 C CNN
 F 3 "~" H 1450 1800 50  0001 C CNN
@@
 	1    0    0    -1
 $EndComp
-Connection ~ 1950 2850
-Wire Wire Line
-	1950 2850 1950 3250
+Connection ~ 1550 2850
+Wire Wire Line
+	1550 2850 1550 3250
 $Comp
 L 74xx:74HC04 INV1
@@
 F34 "WR#" I T 3350 4600 50
 F35 "RD#" I T 3250 4600 50
-F36 "CLK" I T 2950 4600 50
-F37 "RES#" I T 3050 4600 50
+F36 "RES#" I T 3050 4600 50
+F37 "CLKA" I T 2850 4600 50
+F38 "CLKB" I T 2950 4600 50
 $EndSheet
 $Comp
@@
 Wire Wire Line
 	3250 4150 3250 4600
-Wire Wire Line
-	1950 2850 2200 2850
 Connection ~ 3200 1400
 Wire Wire Line
@@
 L 74xx:74HC04 INV1
 U 1 1 60D6D7E8
-P 1650 2850
-F 0 "INV1" H 1650 3167 50  0000 C CNN
-F 1 "74HC04" H 1650 3076 50  0000 C CNN
-F 2 "Package_DIP:DIP-14_W7.62mm" H 1650 2850 50  0001 C CNN
-F 3 "http://www.nxp.com/documents/data_sheet/74HC_HCT04.pdf" H 1650 2850 50  0001 C CNN
-	1    1650 2850
+P 1250 2850
+F 0 "INV1" H 1250 3167 50  0000 C CNN
+F 1 "74HC04" H 1250 3076 50  0000 C CNN
+F 2 "Package_DIP:DIP-14_W7.62mm" H 1250 2850 50  0001 C CNN
+F 3 "http://www.nxp.com/documents/data_sheet/74HC_HCT04.pdf" H 1250 2850 50  0001 C CNN
+	1    1250 2850
 	1    0    0    -1
 $EndComp
@@
 	1    0    0    -1
 $EndComp
-NoConn ~ 2800 4100
 Wire Wire Line
 	2200 3500 2200 4100
 Connection ~ 2200 3500
+$Comp
+L Device:R_POT RV1
+U 1 1 60E14F68
+P 1950 3050
+F 0 "RV1" H 1880 3096 50  0000 R CNN
+F 1 "1k" H 1880 3005 50  0000 R CNN
+F 2 "" H 1950 3050 50  0001 C CNN
+F 3 "~" H 1950 3050 50  0001 C CNN
+	1    1950 3050
+	1    0    0    -1
+$EndComp
+Wire Wire Line
+	1950 2850 1950 2900
+Wire Wire Line
+	1550 2850 1950 2850
+$Comp
+L power:GND #PWR0138
+U 1 1 60E284AB
+P 1950 3300
+F 0 "#PWR0138" H 1950 3050 50  0001 C CNN
+F 1 "GND" H 1955 3127 50  0000 C CNN
+F 2 "" H 1950 3300 50  0001 C CNN
+F 3 "" H 1950 3300 50  0001 C CNN
+	1    1950 3300
+	1    0    0    -1
+$EndComp
+Wire Wire Line
+	1950 3300 1950 3200
+Wire Wire Line
+	2100 3050 2150 3050
+Wire Wire Line
+	2150 3050 2150 2850
+Wire Wire Line
+	2150 2850 2200 2850
+Wire Wire Line
+	2850 4600 2850 4100
+Wire Wire Line
+	2850 4100 2800 4100
 $EndSCHEMATC

Commit message: Rework MMU to use a 74HC138 as in the OS816 reference
Parts:
- removed MMU1: 74HC32, Package_DIP:DIP-14_W7.62mm, symbol 74xx:74LS32
- removed RV1: 1k, symbol Device:R_POT
- added UMMU1: 74HC138, symbol 74xx:74LS138
- renumbered ROM1 to FLASH1
Connections:
- net labels added: CLKFAST, FLASHRD#, FLASHWR#, IORD#, IOWR#, MEM#, RAMRD#, RAMWR#, RWB
- net labels removed: IOSEL#, RAMSEL#, RD#, ROMSEL#, WR#
- wire segments 244 -> 240
- no-connect marks 13 -> 16
Other:
- moved on the sheet: INV1B, INV1C, INV1D, INV1E, INV1F
